Commit message: added colors (works) + add motor/transmission (don't WORK)

File: reflex_description/materials/reflex.gazebo.xacro (robot description, xacro)
@@ -1,10 +1,30 @@
 <?xml version="1.0"?>
 <robot xmlns:xacro="http://www.ros.org/wiki/xacro">
+<!-- Incudes -->
+  <xacro:include filename="$(find reflex_description)/urdf/reflex_takktile_2.xacro" />
+  <xacro:include filename="$(find reflex_description)/urdf/reflex.transmission.xacro" />
+  <!-- Transmissions -->
+  <!-- <xacro:if value="$(arg actuate_reflex)">
+    <xacro:include filename="$(find ll4ma_robots_description)/urdf/reflex/reflex.transmission.xacro"/>
+  </xacro:if> -->
+<!-- Load Gazebo lib and set the robot namespace -->
+    <gazebo>
+      <plugin name="gazebo_ros_control" filename="libgazebo_ros_control.so">
+        <robotNamespace>/reflex_takktile_2</robotNamespace>
+      </plugin>
+    </gazebo>
+    <!-- <gazebo>
+      <plugin name="gazebo_ros_control" filename="libgazebo_ros_control.so">
+        <robotNamespace>rhr_flex_model</robotNamespace>
+        <robotParam>/robot_description</robotParam>
+        <robotSimType>gazebo_ros_control/DefaultRobotHWSim</robotSimType>
+      </plugin>
+    </gazebo> -->
   <!-- materials -->
   <gazebo reference="base_link">
-    <material>Gazebo/Black</material>
+    <material>Gazebo/Green</material>
   </gazebo>
   <gazebo reference="pad">
-    <material>Gazebo/Green</material>
+    <material>Gazebo/FlatBlack</material>
   </gazebo>
   <gazebo reference="swivel_1">
@@ -53,11 +73,11 @@
     <material>Gazebo/FlatBlack</material>
   </gazebo>
-  <gazebo reference="flex_link_1">
+  <gazebo reference="finger_1_flex_link">
     <material>Gazebo/YellowTransparent</material>
   </gazebo>
-  <gazebo reference="flex_link_2">
+  <gazebo reference="finger_2_flex_link">
     <material>Gazebo/YellowTransparent</material>
   </gazebo>
-  <gazebo reference="flex_link_3">
+  <gazebo reference="finger_3_flex_link">
     <material>Gazebo/YellowTransparent</material>
   </gazebo>

File: reflex_description/urdf/reflex_takktile_2.xacro (robot description, xacro)
@@ -3,4 +3,8 @@
    01.05.2019 -->
 <robot name="reflex_takktile_2" xmlns:xacro="http://ros.org/wiki/xacro">
+<!-- Incudes -->
+  <!-- <xacro:include filename="$(find reflex_description)/urdf/reflex.transmission.xacro" /> -->
+  <!-- <xacro:include filename="$(find reflex_description)/materials/reflex.gazebo.xacro" /> -->
+  <xacro:include filename="$(find reflex_description)/materials/reflex.materials.xacro" />
 <!-- Properties -->
   <xacro:property name="flex_link_mass"     value="0.01"/>
@@ -19,5 +23,5 @@
   <xacro:property name="prox_length" value="0.060" />
   <xacro:property name="pi" value="3.1415" />
-  <xacro:macro name="base_color">
+  <!-- <xacro:macro name="base_color">
     <color rgba="0.1 0.1 0.1 1"/>
   </xacro:macro>
@@ -39,5 +43,5 @@
   <material name="orange">
     <color rgba="${255/255} ${108/255} ${10/255} 1.0"/>
-  </material>
+  </material> -->
 <!-- ################ ################ ################ ################ ################ ################ -->
 <!-- ################ THE SECTION CREATED BY SOLIDWORKS EXPORTER, CUT AND PASTE THIS IN HERE ################ -->
