Commit message: Finger 1 done

File: reflex_description/materials/reflex.materials.xacro (robot description, xacro)
@@ -6,6 +6,6 @@
   </xacro:if> -->
   <!-- materials -->
-  <gazebo reference="lower_shell">
-    <material>Gazebo/Black</material>
+  <gazebo reference="base_link">
+    <material>Gazebo/Green</material>
   </gazebo>
   <gazebo reference="pad">

File: reflex_description/urdf/reflex_takktile_2.xacro (robot description, xacro)
@@ -3,5 +3,4 @@
    01.05.2019 -->
 <robot name="reflex_takktile_2" xmlns:xacro="http://ros.org/wiki/xacro">
- <!-- <robot name="robot_test" xmlns:xacro="http://ros.org/wiki/xacro"> -->
 <!-- Properties -->
   <xacro:property name="flex_link_mass"     value="0.01"/>
@@ -38,4 +37,7 @@
     <color rgba="0.2 0.8 0.75 1"/>
   </xacro:macro>
+  <material name="orange">
+    <color rgba="${255/255} ${108/255} ${10/255} 1.0"/>
+  </material>
 <!-- ################ ################ ################ ################ ################ ################ -->
 <!-- ################ THE SECTION CREATED BY SOLIDWORKS EXPORTER, CUT AND PASTE THIS IN HERE ################ -->
@@ -48,5 +50,5 @@
       <origin xyz="0.0 0.0 0.0"/>
       <!-- TODO: CALCULATES THE MASS AND INERTIAs -->
-      <mass value="0.7"/>
+      <mass value="${base_link_mass}"/>
       <inertia
         ixx="0.0001" ixy="0.0" ixz="0.0"
@@ -285,4 +287,5 @@
     </inertial>
     <visual>
+      <!-- <origin xyz="-0.077 0.007 0.007" rpy="3.1459 0 0" /> -->
       <origin xyz="-0.077 0.007 0.007" rpy="3.1459 0 0" />
       <!-- <origin xyz="0.0 0.0 0.0" rpy="3.1459 0 0" /> -->
@@ -298,5 +301,4 @@
     <collision>
       <origin xyz="-0.077 0.007 0.007" rpy="3.1459 0 0" />
-      <!-- <origin xyz="0.0 0.0 0.0" rpy="3.1459 0 0" /> -->
       <geometry>
         <mesh filename="package://reflex_description/meshes/distal_1.STL" />
@@ -319,5 +321,5 @@
     <!-- <origin xyz="${flex_length-0.01} 0 0.008" rpy="0 0 0" /> -->
     <!-- <origin xyz="${flex_length-0.01} 0 0.000" rpy="0 0 0" /> -->
-    <origin xyz="0.0 0 0.0" rpy="0 0 0" />
+    <origin xyz="${flex_length-0.01} 0 0.001" rpy="0 0 0" />
     <parent link="flex_link_1" />
     <child link="distal_1" />
@@ -327,7 +329,5 @@
   <link name="distal_pad_1">
     <inertial>
-      <!-- TODO: CALCULATES CENTER OF MASS -->
-      <origin xyz="0.0 0.0 0.0"/>
-      <!-- TODO: CALCULATES THE MASS AND INERTIAs -->
+      <origin xyz="0.0 0.0 0.0"/>
       <mass value="0.01"/>
       <inertia
@@ -506,4 +506,5 @@
     </visual>
   </link>
+<!-- *****************************************FINGER 3**************************************************** -->
   <joint name="proximal_joint_3" type="continuous">
     <origin

Commit message: moved files.

File: reflex_description/materials/reflex.materials.xacro (robot description, xacro)
@@ -1,4 +1,8 @@
 <?xml version="1.0"?>
 <robot xmlns:xacro="http://www.ros.org/wiki/xacro">
+  <!-- Incudes -->
+  <!-- <xacro:include filename="$(find reflex_description)/urdf/reflex.transmission.xacro" /> -->
+  <!-- <xacro:include filename="$(find reflex_description)/urdf/reflex.gazebo.xacro" /> -->
+  <xacro:include filename="$(find reflex_description)/urdf/reflex_takktile_2.xacro" />
   <!-- materials -->
   <gazebo reference="base_link">

File: reflex_description/urdf/reflex.transmission.xacro (robot description, xacro)
@@ -3,5 +3,6 @@
 <!-- Incudes -->
   <xacro:include filename="$(find reflex_description)/urdf/reflex_takktile_2.xacro" />
-  <!-- <xacro:include filename="$(find reflex_description)/materials/reflex.gazebo.xacro" /> -->
+  <!-- <xacro:include filename="$(find reflex_description)/urdf/reflex.gazebo.xacro" /> -->
+  <xacro:include filename="$(find reflex_description)/materials/reflex.materials.xacro" />
 <!-- Transmission -->
   <transmission name="preshape_transmission_1">

File: reflex_description/urdf/reflex_takktile_2.xacro (robot description, xacro)
@@ -5,5 +5,5 @@
 <!-- Incudes -->
   <!-- <xacro:include filename="$(find reflex_description)/urdf/reflex.transmission.xacro" /> -->
-  <!-- <xacro:include filename="$(find reflex_description)/materials/reflex.gazebo.xacro" /> -->
+  <!-- <xacro:include filename="$(find reflex_description)/urdf/reflex.gazebo.xacro" /> -->
   <xacro:include filename="$(find reflex_description)/materials/reflex.materials.xacro" />
 <!-- Properties -->
@@ -23,25 +23,4 @@
   <xacro:property name="prox_length" value="0.060" />
   <xacro:property name="pi" value="3.1415" />
-  <!-- <xacro:macro name="base_color">
-    <color rgba="0.1 0.1 0.1 1"/>
-  </xacro:macro>
-  <xacro:macro name="swivel_color">
-    <color rgba="0.1 0.1 0.1 1"/>
-  </xacro:macro>
-  <xacro:macro name="proximal_color">
-    <color rgba="0.16 0.16 0.16 1"/>
-  </xacro:macro>
-   <xacro:macro name="distal_color">
-    <color rgba="0.16 0.16 0.16 1"/>
-  </xacro:macro>
-  <xacro:macro name="flex_color">
-    <color rgba="0.2 0.2 .2 1"/>
-  </xacro:macro>
-  <xacro:macro name="pad_color">
-    <color rgba="0.2 0.8 0.75 1"/>
-  </xacro:macro>
-  <material name="orange">
-    <color rgba="${255/255} ${108/255} ${10/255} 1.0"/>
-  </material> -->
 <!-- ################ ################ ################ ################ ################ ################ -->
 <!-- ################ THE SECTION CREATED BY SOLIDWORKS EXPORTER, CUT AND PASTE THIS IN HERE ################ -->

Commit message: set effort

File: reflex_description/materials/reflex.materials.xacro (robot description, xacro)
@@ -23,4 +23,6 @@
   <gazebo reference="distal_1">
     <material>Gazebo/FlatBlack</material>
+    <mu1>0.2</mu1>
+    <mu2>0.2</mu2>
   </gazebo>
   <gazebo reference="distal_2">

File: reflex_description/urdf/reflex_takktile_2.xacro (robot description, xacro)
@@ -18,13 +18,13 @@
 <!-- Parameters joints -->
   <!-- Preshape -->
+  <xacro:property name="preshape_joint_limit_effort"     value="1.0"/>
+  <xacro:property name="preshape_joint_limit_velocity"   value="1.0"/>
   <xacro:property name="preshape_joint_limit_lower"      value="-0.0872665"/>
   <xacro:property name="preshape_joint_limit_upper"      value="2.09440"/>
-  <xacro:property name="preshape_joint_limit_velocity"   value="1.0"/>
-  <xacro:property name="preshape_joint_limit_effort"     value="30.0"/>
   <!-- Proximal -->
+  <xacro:property name="proximal_joint_limit_effort"     value="1.0"/>
+  <xacro:property name="proximal_joint_limit_velocity"   value="1.0"/>
   <xacro:property name="proximal_joint_limit_lower"      value="0.0"/>
   <xacro:property name="proximal_joint_limit_upper"      value="2.09440"/>
-  <xacro:property name="proximal_joint_limit_velocity"   value="1.0"/>
-  <xacro:property name="proximal_joint_limit_effort"     value="30.0"/>
 <!-- ################ ################ ################ ################ ################ ################ -->
 <!-- ################ XACRO PORTION OF THE URDF, FOR MAKING THE FLEXIBLE JOINTS ################ -->
