Commit message: repair the broken code... everything work

File: reflex_description/urdf/reflex.transmission.xacro (robot description, xacro)
@@ -6,5 +6,6 @@
   <!-- <xacro:include filename="$(find reflex_description)/materials/reflex.materials.xacro" /> -->
 <!-- Transmission -->
-  <transmission name="preshape_transmission_1">
+<!-- Preshape -->
+  <transmission name="preshape_1_transmission">
     <type>transmission_interface/SimpleTransmission</type>
     <joint name="preshape_1">
@@ -15,4 +16,4 @@
       <mechanicalReduction>1</mechanicalReduction>
     </actuator>
-</transmission>
+  </transmission>
 </robot>

File: reflex_description/urdf/reflex_takktile_2.xacro (robot description, xacro)
@@ -100,5 +100,5 @@
       xyz="0 0 0" />
   </joint>
-  <!-- *****************************************FINGER 1**************************************************** -->
+<!-- *****************************************FINGER 1**************************************************** -->
   <link name="swivel_1">
     <inertial>
@@ -290,5 +290,5 @@
     </collision>
   </link>
-  <joint name="distal_joint_1"  type="continuous">
+  <joint name="distal_joint_1"  type="fixed">
     <!-- type="revolute"> -->
     <!-- type="continuous"> -->
@@ -344,5 +344,5 @@
     <axis xyz="0 0 0" />
   </joint>
-  <!-- *****************************************FINGER 2**************************************************** -->
+<!-- *****************************************FINGER 2**************************************************** -->
   <link name="swivel_2">
     <inertial>
@@ -536,5 +536,5 @@
     </collision>
   </link>
-  <joint name="distal_joint_2" type="continuous">
+  <joint name="distal_joint_2" type="fixed">
     <origin xyz="${flex_length-0.01} 0 0.001" rpy="0 0 0" />
     <parent
@@ -733,5 +733,5 @@
     </collision>
   </link>
-  <joint name="distal_joint_3" type="continuous">
+  <joint name="distal_joint_3" type="fixed">
     <origin xyz="${flex_length-0.01} 0 0.001" rpy="0 0 0" />
     <parent

Commit message: add the proximal motor

File: reflex_description/urdf/reflex.transmission.xacro (robot description, xacro)
@@ -17,3 +17,44 @@
     </actuator>
   </transmission>
+  <transmission name="preshape_2_transmission">
+    <type>transmission_interface/SimpleTransmission</type>
+    <joint name="preshape_2">
+      <hardwareInterface>EffortJointInterface</hardwareInterface>
+    </joint>
+    <actuator name="preshape_2_motor">
+      <hardwareInterface>EffortJointInterface</hardwareInterface>
+      <mechanicalReduction>1</mechanicalReduction>
+    </actuator>
+  </transmission>
+<!-- Proximal -->
+  <transmission name="proximal_1_transmission">
+    <type>transmission_interface/SimpleTransmission</type>
+    <joint name="proximal_joint_1">
+      <hardwareInterface>EffortJointInterface</hardwareInterface>
+    </joint>
+    <actuator name="proximal_1_motor">
+      <hardwareInterface>EffortJointInterface</hardwareInterface>
+      <mechanicalReduction>1</mechanicalReduction>
+    </actuator>
+  </transmission>
+  <transmission name="proximal_2_transmission">
+    <type>transmission_interface/SimpleTransmission</type>
+    <joint name="proximal_joint_2">
+      <hardwareInterface>EffortJointInterface</hardwareInterface>
+    </joint>
+    <actuator name="proximal_2_motor">
+      <hardwareInterface>EffortJointInterface</hardwareInterface>
+      <mechanicalReduction>1</mechanicalReduction>
+    </actuator>
+  </transmission>
+  <transmission name="proximal_3_transmission">
+    <type>transmission_interface/SimpleTransmission</type>
+    <joint name="proximal_joint_3">
+      <hardwareInterface>EffortJointInterface</hardwareInterface>
+    </joint>
+    <actuator name="proximal_3_motor">
+      <hardwareInterface>EffortJointInterface</hardwareInterface>
+      <mechanicalReduction>1</mechanicalReduction>
+    </actuator>
+  </transmission>
 </robot>
