Commit message: add the hand to an hand effector

File: reflex_description/urdf/reflex_takktile_2_tool.xacro (robot description, xacro)
@@ -80,9 +80,9 @@
   </link>
   <!-- For a tool on a arm, uncomment this part -->
-  <!-- <joint name="tool_joint" type="fixed">
+  <joint name="tool_joint" type="fixed">
       <parent link="iiwa_link_ee" />
       <child link = "base_link" />
       <origin xyz="0.0 0.0 0.0" rpy="0 0.0 3.14159" />
-  </joint> -->
+  </joint>
   <link name="pad">
     <inertial>
