Commit message: Add the plugin contact and it works but I have to publish the message through ros and then add the 9 sensors per finger

File: reflex_description/urdf/reflex.gazebo.xacro (robot description, xacro)
@@ -9,17 +9,27 @@
   </xacro:if> -->
 <!-- Load Gazebo lib and set the robot namespace -->
-    <gazebo>
-      <plugin name="gazebo_ros_control" filename="libgazebo_ros_control.so">
-        <robotNamespace>reflex_takktile_2</robotNamespace>
-        <robotParam>/robot_description</robotParam>
-        <robotSimType>gazebo_ros_control/DefaultRobotHWSim</robotSimType>
-      </plugin>
-    </gazebo>
-    <!-- <gazebo>
-      <plugin name="gazebo_ros_control" filename="libgazebo_ros_control.so">
-        <robotNamespace>rhr_flex_model</robotNamespace>
-        <robotParam>/robot_description</robotParam>
-        <robotSimType>gazebo_ros_control/DefaultRobotHWSim</robotSimType>
-      </plugin>
-    </gazebo> -->
+  <gazebo>
+    <plugin name="gazebo_ros_control" filename="libgazebo_ros_control.so">
+      <robotNamespace>reflex_takktile_2</robotNamespace>
+      <robotParam>/robot_description</robotParam>
+      <robotSimType>gazebo_ros_control/DefaultRobotHWSim</robotSimType>
+    </plugin>
+  </gazebo>
+  <!-- <gazebo>
+    <sensor name="finger_1_sensor_1" type="contact">
+    <plugin name="my_plugin" filename="libcontact.so"/>
+      <contact>
+        <collision>proximal_pad_1_collision</collision>
+      </contact>
+    </sensor>
+  </gazebo> -->
+  <gazebo reference="proximal_pad_1">
+    <sensor name='proximal_pad_1_contact_sensor' type='contact'>
+      <plugin name="proximal_pad_1_contact_sensor_plugin" filename="libcontact.so"/>
+          <contact>
+            <collision>proximal_pad_1_collision</collision>
+          </contact>
+      <update_rate>30</update_rate>
+    </sensor>
+  </gazebo>
 </robot>

File: reflex_description/urdf/reflex_takktile_2.xacro (robot description, xacro)
@@ -219,5 +219,5 @@
       </material>
     </visual>
-    <collision>
+    <collision name="proximal_pad_1_collision">
       <origin xyz="-0.008 0.014 -0.002" rpy="1.5708 1.5708 0" />
       <geometry>

Commit message: everything works until here (compilation, build + roslaunch)

File: reflex_description/urdf/reflex.gazebo.xacro (robot description, xacro)
@@ -16,13 +16,6 @@
     </plugin>
   </gazebo>
-  <!-- <gazebo>
-    <sensor name="finger_1_sensor_1" type="contact">
-    <plugin name="my_plugin" filename="libcontact.so"/>
-      <contact>
-        <collision>proximal_pad_1_collision</collision>
-      </contact>
-    </sensor>
-  </gazebo> -->
-  <gazebo reference="proximal_pad_1">
+  <!-- Keep for souvenir -->
+  <!-- <gazebo reference="proximal_pad_1">
     <sensor name='proximal_pad_1_contact_sensor' type='contact'>
       <plugin name="proximal_pad_1_contact_sensor_plugin" filename="libcontact.so"/>
@@ -32,4 +25,26 @@
       <update_rate>30</update_rate>
     </sensor>
-  </gazebo>
+  </gazebo> -->
+  <!-- Proximal  -->
+  <!-- 5 sensors on the proximal -->
+  <!-- <gazebo reference="proximal_1_sensor_1">
+    <sensor name='proximal_1_contact_sensor_1' type='contact'>
+      <plugin name="proximal_1_contact_sensor_1_plugin" filename="libcontact.so"/>
+          <contact>
+            <collision>proximal_1_sensor_1_collision</collision>
+          </contact>
+      <update_rate>30</update_rate>
+    </sensor>
+  </gazebo> -->
+  <!-- Distal -->
+  <!-- 4 sensors on the distal -->
+  <!-- <gazebo reference="distal_1_sensor_1">
+    <sensor name='distal_1_contact_sensor_1' type='contact'>
+      <plugin name="distal_1_contact_sensor_1_plugin" filename="libcontact.so"/>
+          <contact>
+            <collision>distal_1_sensor_1_collision</collision>
+          </contact>
+      <update_rate>30</update_rate>
+    </sensor>
+  </gazebo> -->
 </robot>

File: reflex_description/urdf/reflex_takktile_2.xacro (robot description, xacro)
@@ -219,5 +219,12 @@
       </material>
     </visual>
-    <collision name="proximal_pad_1_collision">
+    <!-- Keep for souvenir -->
+    <!-- <collision name="proximal_pad_1_collision">
+      <origin xyz="-0.008 0.014 -0.002" rpy="1.5708 1.5708 0" />
+      <geometry>
+        <mesh filename="package://reflex_description/meshes/proximal_pad_1.STL" />
+      </geometry>
+    </collision> -->
+    <collision>
       <origin xyz="-0.008 0.014 -0.002" rpy="1.5708 1.5708 0" />
       <geometry>

Commit message: add the tactile sensor on the hand

File: reflex_description/urdf/reflex.gazebo.xacro (robot description, xacro)
@@ -37,4 +37,30 @@
     </sensor>
   </gazebo> -->
+  <xacro:macro name="proximal_sensor_gazebo_macro" params="finger_number sensor_number">
+    <gazebo reference="proximal_${finger_number}_sensor_${sensor_number}">
+      <sensor name='proximal_${finger_number}_sensor_${sensor_number}_contact_sensor' type='contact'>
+        <plugin name="proximal_${finger_number}_sensor_${sensor_number}_contact_sensor_plugin" filename="libcontact.so"/>
+            <contact>
+              <collision>proximal_${finger_number}_sensor_${sensor_number}_collision</collision>
+            </contact>
+        <update_rate>30</update_rate>
+      </sensor>
+    </gazebo>
+  </xacro:macro>
+  <xacro:proximal_sensor_gazebo_macro finger_number="1" sensor_number="1"/>
+  <xacro:proximal_sensor_gazebo_macro finger_number="1" sensor_number="2"/>
+  <xacro:proximal_sensor_gazebo_macro finger_number="1" sensor_number="3"/>
+  <xacro:proximal_sensor_gazebo_macro finger_number="1" sensor_number="4"/>
+  <xacro:proximal_sensor_gazebo_macro finger_number="1" sensor_number="5"/>
+  <xacro:proximal_sensor_gazebo_macro finger_number="2" sensor_number="1"/>
+  <xacro:proximal_sensor_gazebo_macro finger_number="2" sensor_number="2"/>
+  <xacro:proximal_sensor_gazebo_macro finger_number="2" sensor_number="3"/>
+  <xacro:proximal_sensor_gazebo_macro finger_number="2" sensor_number="4"/>
+  <xacro:proximal_sensor_gazebo_macro finger_number="2" sensor_number="5"/>
+  <xacro:proximal_sensor_gazebo_macro finger_number="3" sensor_number="1"/>
+  <xacro:proximal_sensor_gazebo_macro finger_number="3" sensor_number="2"/>
+  <xacro:proximal_sensor_gazebo_macro finger_number="3" sensor_number="3"/>
+  <xacro:proximal_sensor_gazebo_macro finger_number="3" sensor_number="4"/>
+  <xacro:proximal_sensor_gazebo_macro finger_number="3" sensor_number="5"/>
   <!-- Distal -->
   <!-- 4 sensors on the distal -->
@@ -48,3 +74,26 @@
     </sensor>
   </gazebo> -->
+  <xacro:macro name="distal_sensor_gazebo_macro" params="finger_number sensor_number">
+    <gazebo reference="distal_${finger_number}_sensor_${sensor_number}">
+      <sensor name='distal_${finger_number}_sensor_${sensor_number}_contact_sensor' type='contact'>
+        <plugin name="distal_${finger_number}_sensor_${sensor_number}_contact_sensor_plugin" filename="libcontact.so"/>
+            <contact>
+              <collision>distal_${finger_number}_sensor_${sensor_number}_collision</collision>
+            </contact>
+        <update_rate>30</update_rate>
+      </sensor>
+    </gazebo>
+  </xacro:macro>
+  <xacro:distal_sensor_gazebo_macro finger_number="1" sensor_number="1"/>
+  <xacro:distal_sensor_gazebo_macro finger_number="1" sensor_number="2"/>
+  <xacro:distal_sensor_gazebo_macro finger_number="1" sensor_number="3"/>
+  <xacro:distal_sensor_gazebo_macro finger_number="1" sensor_number="4"/>
+  <xacro:distal_sensor_gazebo_macro finger_number="2" sensor_number="1"/>
+  <xacro:distal_sensor_gazebo_macro finger_number="2" sensor_number="2"/>
+  <xacro:distal_sensor_gazebo_macro finger_number="2" sensor_number="3"/>
+  <xacro:distal_sensor_gazebo_macro finger_number="2" sensor_number="4"/>
+  <xacro:distal_sensor_gazebo_macro finger_number="3" sensor_number="1"/>
+  <xacro:distal_sensor_gazebo_macro finger_number="3" sensor_number="2"/>
+  <xacro:distal_sensor_gazebo_macro finger_number="3" sensor_number="3"/>
+  <xacro:distal_sensor_gazebo_macro finger_number="3" sensor_number="4"/>
 </robot>

File: reflex_description/urdf/reflex_takktile_2.xacro (robot description, xacro)
@@ -7,4 +7,5 @@
   <xacro:include filename="$(find reflex_description)/urdf/reflex.gazebo.xacro" />
   <xacro:include filename="$(find reflex_description)/materials/reflex.materials.xacro" />
+  <xacro:include filename="$(find reflex_description)/urdf/tactile_sensors.xacro" />
 <!-- Properties -->
   <xacro:property name="flex_link_mass"     value="0.01"/>
@@ -31,4 +32,5 @@
 <!-- ################ ################ ################ ################ ################ ################ -->
   <xacro:property name="flex_length" value="0.016" />
+  <xacro:property name="distal_length" value="0.050" />
   <xacro:property name="num_steps" value="9" />
   <xacro:property name="prox_length" value="0.060" />
@@ -811,5 +813,5 @@
 <!-- ################ COPY AND PASTE THIS FROM urdf/homemade_marker_portion_urdf  ################ -->
 <!-- ################ ################ ################ ################ ################ ################ -->
-  <joint name="base_tactile_joint" type="fixed">
+  <!-- <joint name="base_tactile_joint" type="fixed">
     <origin xyz="0 0 0" rpy="0 0 0" />
     <parent link="base_link" />
@@ -852,4 +854,33 @@
     <child link="distal_3_tactile" />
   </joint>
-  <link name="distal_3_tactile"/>
+  <link name="distal_3_tactile"/> -->
+  <!-- Tactile sensors -->
+  <!-- Example -->
+  <!-- <collision name="proximal_pad_1_collision">
+      <origin xyz="-0.008 0.014 -0.002" rpy="1.5708 1.5708 0" />
+      <geometry>
+        <mesh filename="package://reflex_description/meshes/proximal_pad_1.STL" />
+      </geometry>
+    </collision> -->
+  <!-- <link name="proximal_1_sensor_1">
+    <inertial>
+      <mass value="0.00001"/>
+      <inertia
+        ixx="0.00000000001" ixy="0.0" ixz="0.0"
+                        iyy="0.00000000001"  iyz="0.0"
+                                          izz="0.00000000001"/>
+    </inertial>
+    <visual>
+      <origin xyz="0 0 0" rpy="0 0.0 0" />
+      <geometry>
+        <cylinder length="0.002" radius="0.004"/>
+      </geometry>
+    </visual>
+    <collision>
+      <origin xyz="0 0 0.0" rpy="0 0.0 0" />
+      <geometry>
+        <cylinder length="0.002" radius="0.004"/>
+      </geometry>
+    </collision>
+  </link> -->
 </robot>

Commit message: add the motor

File: reflex_description/urdf/reflex.gazebo.xacro (robot description, xacro)
@@ -4,8 +4,4 @@
   <!-- <xacro:include filename="$(find reflex_description)/urdf/reflex_takktile_2.xacro" />
   <xacro:include filename="$(find reflex_description)/urdf/reflex.transmission.xacro" /> -->
-  <!-- Transmissions -->
-  <!-- <xacro:if value="$(arg actuate_reflex)">
-    <xacro:include filename="$(find ll4ma_robots_description)/urdf/reflex/reflex.transmission.xacro"/>
-  </xacro:if> -->
 <!-- Load Gazebo lib and set the robot namespace -->
   <gazebo>
@@ -16,14 +12,4 @@
     </plugin>
   </gazebo>
-  <!-- Keep for souvenir -->
-  <!-- <gazebo reference="proximal_pad_1">
-    <sensor name='proximal_pad_1_contact_sensor' type='contact'>
-      <plugin name="proximal_pad_1_contact_sensor_plugin" filename="libcontact.so"/>
-          <contact>
-            <collision>proximal_pad_1_collision</collision>
-          </contact>
-      <update_rate>30</update_rate>
-    </sensor>
-  </gazebo> -->
   <!-- Proximal  -->
   <!-- 5 sensors on the proximal -->

File: reflex_description/urdf/reflex.transmission.xacro (robot description, xacro)
@@ -58,3 +58,34 @@
     </actuator>
   </transmission>
+  <!-- Distal -->
+  <transmission name="distal_1_transmission">
+    <type>transmission_interface/SimpleTransmission</type>
+    <joint name="distal_joint_1">
+      <hardwareInterface>EffortJointInterface</hardwareInterface>
+    </joint>
+    <actuator name="distal_1_motor">
+      <hardwareInterface>EffortJointInterface</hardwareInterface>
+      <mechanicalReduction>1</mechanicalReduction>
+    </actuator>
+  </transmission>
+  <transmission name="distal_2_transmission">
+    <type>transmission_interface/SimpleTransmission</type>
+    <joint name="distal_joint_2">
+      <hardwareInterface>EffortJointInterface</hardwareInterface>
+    </joint>
+    <actuator name="distal_2_motor">
+      <hardwareInterface>EffortJointInterface</hardwareInterface>
+      <mechanicalReduction>1</mechanicalReduction>
+    </actuator>
+  </transmission>
+  <transmission name="distal_3_transmission">
+    <type>transmission_interface/SimpleTransmission</type>
+    <joint name="distal_joint_3">
+      <hardwareInterface>EffortJointInterface</hardwareInterface>
+    </joint>
+    <actuator name="distal_3_motor">
+      <hardwareInterface>EffortJointInterface</hardwareInterface>
+      <mechanicalReduction>1</mechanicalReduction>
+    </actuator>
+  </transmission>
 </robot>

File: reflex_description/urdf/reflex_takktile_2.xacro (robot description, xacro)
@@ -12,6 +12,4 @@
   <xacro:include filename="$(find reflex_description)/materials/reflex.materials.xacro" />
   <xacro:include filename="$(find reflex_description)/urdf/tactile_sensors.xacro" />
-  <xacro:include filename="$(find iiwa_description)/urdf/iiwa7.xacro"/>
-  <xacro:include filename="$(find iiwa_description)/urdf/iiwa7.urdf.xacro"/>
 <!-- Properties -->
   <xacro:property name="flex_link_mass"     value="0.01"/>
@@ -23,5 +21,5 @@
   <xacro:property name="base_link_mass"     value="0.74"/>
   <xacro:property name="pad_mass"           value="0.1"/>
-<!-- Parameters joints -->
+<!-- Parameters Limits Joints -->
   <!-- Preshape -->
   <xacro:property name="preshape_joint_limit_effort"     value="1.0"/>
@@ -34,4 +32,9 @@
   <xacro:property name="proximal_joint_limit_lower"      value="0.0"/>
   <xacro:property name="proximal_joint_limit_upper"      value="2.09440"/>
+  <!-- Distal -->
+  <xacro:property name="distal_joint_limit_effort"     value="1.0"/>
+  <xacro:property name="distal_joint_limit_velocity"   value="1.0"/>
+  <xacro:property name="distal_joint_limit_lower"      value="0.0"/>
+  <xacro:property name="distal_joint_limit_upper"      value="1.8"/>
 <!-- ################ ################ ################ ################ ################ ################ -->
 <!-- ################ XACRO PORTION OF THE URDF, FOR MAKING THE FLEXIBLE JOINTS ################ -->
@@ -325,24 +328,13 @@
     </collision>
   </link>
-  <joint name="distal_joint_1"  type="fixed">
-    <!-- type="revolute"> -->
-    <!-- type="continuous"> -->
-    <!-- <origin
-      xyz="0.07600000000000001 0 0.00250000000000002"
-      rpy="0 0 0" />
-    <parent
-      link="proximal_1" />
-    <child
-      link="distal_1" />
-    <axis
-      xyz="0 -1 0" /> -->
-    <!-- <origin xyz="${flex_length} 0 0.00250000000000002" rpy="0 0 0" /> -->
-    <!-- <origin xyz="${flex_length-0.01} 0 0.008" rpy="0 0 0" /> -->
-    <!-- <origin xyz="${flex_length-0.01} 0 0.000" rpy="0 0 0" /> -->
+  <joint name="distal_joint_1"  type="revolute">
     <origin xyz="${flex_length-0.01} 0 0.001" rpy="0 0 0" />
     <parent link="flex_link_1" />
     <child link="distal_1" />
     <axis xyz="0 -1 0" />
-    <!-- <limit effort="0.25" velocity="1.0" lower="0" upper="2.74" /> -->
+    <limit effort="${distal_joint_limit_effort}"
+            velocity="${distal_joint_limit_velocity}"
+            lower="${distal_joint_limit_lower}"
+            upper="${distal_joint_limit_upper}" />
   </joint>
   <link name="distal_pad_1">
@@ -574,12 +566,14 @@
     </collision>
   </link>
-  <joint name="distal_joint_2" type="fixed">
+  <joint name="distal_joint_2" type="revolute">
     <origin xyz="${flex_length-0.01} 0 0.001" rpy="0 0 0" />
     <parent
       link="flex_link_2" />
-    <child
-      link="distal_2" />
-    <axis
-      xyz="0 -1 0" />
+    <child link="distal_2" />
+    <axis xyz="0 -1 0" />
+      <limit effort="${distal_joint_limit_effort}"
+            velocity="${distal_joint_limit_velocity}"
+            lower="${distal_joint_limit_lower}"
+            upper="${distal_joint_limit_upper}" />
   </joint>
   <link name="distal_pad_2">
@@ -772,12 +766,14 @@
     </collision>
   </link>
-  <joint name="distal_joint_3" type="fixed">
+  <joint name="distal_joint_3" type="revolute">
     <origin xyz="${flex_length-0.01} 0 0.001" rpy="0 0 0" />
     <parent
       link="flex_link_3" />
-    <child
-      link="distal_3" />
-    <axis
-      xyz="0 -1 0" />
+    <child link="distal_3" />
+    <axis xyz="0 -1 0" />
+      <limit effort="${distal_joint_limit_effort}"
+            velocity="${distal_joint_limit_velocity}"
+            lower="${distal_joint_limit_lower}"
+            upper="${distal_joint_limit_upper}" />
   </joint>
   <link name="distal_pad_3">

Commit message: add the hand controller

File: reflex_description/urdf/reflex.gazebo.xacro (robot description, xacro)
@@ -83,3 +83,27 @@
   <xacro:distal_sensor_gazebo_macro finger_number="3" sensor_number="3"/>
   <xacro:distal_sensor_gazebo_macro finger_number="3" sensor_number="4"/>
+  <gazebo reference="$distal_pad_1">
+      <kp>1000000.0</kp>
+      <kd>100.0</kd>
+      <mu1>1.0</mu1>
+      <mu2>1.0</mu2>
+      <maxVel>1.0</maxVel>
+			<!-- <maxContacts>1</maxContacts> -->
+  </gazebo>
+  <gazebo reference="$distal_pad_2">
+      <kp>1000000.0</kp>
+      <kd>100.0</kd>
+      <mu1>1.0</mu1>
+      <mu2>1.0</mu2>
+      <maxVel>1.0</maxVel>
+			<!-- <maxContacts>1</maxContacts> -->
+  </gazebo>
+  <gazebo reference="$distal_pad_3">
+      <kp>1000000.0</kp>
+      <kd>100.0</kd>
+      <mu1>1.0</mu1>
+      <mu2>1.0</mu2>
+      <maxVel>1.0</maxVel>
+			<!-- <maxContacts>1</maxContacts> -->
+  </gazebo>
 </robot>

File: reflex_description/urdf/reflex_takktile_2.xacro (robot description, xacro)
@@ -395,4 +395,18 @@
     </visual>
     <collision>
+      <!-- <surface>
+        <friction>
+          <ode>
+            <mu>100.0</mu>
+            <mu2>100.0</mu2>
+          </ode>
+        </friction>
+        <contact>
+          <ode>
+            <min_depth>0.003</min_depth>
+            <maxVel>0</maxVel>
+          </ode>
+        </contact>
+      </surface> -->
       <origin xyz="-0.00825 0.009 0.057" rpy="1.5708 1.5708 0" />
       <geometry>
@@ -635,4 +649,19 @@
     </visual>
     <collision>
+      <!-- <surface>
+        <surface>
+        <friction>
+          <ode>
+            <mu>100.0</mu>
+            <mu2>100.0</mu2>
+          </ode>
+        </friction>
+        <contact>
+          <ode>
+            <min_depth>0.003</min_depth>
+            <maxVel>0</maxVel>
+          </ode>
+        </contact>
+      </surface> -->
       <origin xyz="-0.00825 0.009 0.057" rpy="1.5708 1.5708 0" />
       <geometry>
@@ -836,4 +865,18 @@
     </visual>
     <collision>
+      <!-- <surface>
+        <friction>
+          <ode>
+            <mu>100.0</mu>
+            <mu2>100.0</mu2>
+          </ode>
+        </friction>
+        <contact>
+          <ode>
+            <min_depth>0.003</min_depth>
+            <maxVel>0</maxVel>
+          </ode>
+        </contact>
+      </surface> -->
       <origin xyz="-0.00825 0.009 0.057" rpy="1.5708 1.5708 0" />
       <geometry>
@@ -853,4 +896,34 @@
       xyz="0 0 0" />
   </joint>
+<!-- ******************************************************************************************************* -->
+<!-- Objects to drop -->
+<!-- ******************************************************************************************************* -->
+  <!-- <link name="square">
+    <inertial>
+      <origin xyz="0.0 0.0 0.0"/>
+      <mass value="0.5"/>
+      <inertia
+        ixx="0.0001" ixy="0.0" ixz="0.0"
+                         iyy="0.0001"  iyz="0.0"
+                                           izz="0.0001"/>
+    </inertial>
+    <visual>
+      <origin
+        xyz="0 0 0" rpy="0 0 0" />
+      <geometry>
+        <box size="0.05 0.05 0.05"/>
+      </geometry>
+      <material
+        name="base_color">
+        <xacro:base_color/>
+      </material>
+    </visual>
+    <collision>
+      <origin xyz="0.0 0.0 0.0" rpy="0 0 0" />
+      <geometry>
+        <box size="0.05 0.05 0.05"/>
+      </geometry>
+    </collision>
+  </link> -->
 <!-- ################ ################ ################ ################ ################ ################ -->
 <!-- ################ THIS SECTION LINKS THE MARKERS (TACTILE DATA) TO THE CAD MESH ################ -->
