Commit message: start the urdf and gazebo simulation of the hand

File: reflex_description/urdf/reflex_takktile_2.xacro (robot description, xacro)
@@ -1,4 +1,16 @@
 <?xml version="1.0"?>
-<robot xmlns:xacro="http://www.ros.org/wiki/xacro" name="rhr_flex_model">
+<!-- Jonathan Burkhard, ETH Zurich, Switzerland
+   01.05.2019 -->
+<robot name="reflex_takktile_2" xmlns:xacro="http://ros.org/wiki/xacro">
+ <!-- <robot name="robot_test" xmlns:xacro="http://ros.org/wiki/xacro"> -->
+<!-- Properties -->
+  <xacro:property name="flex_link_mass"     value="0.01"/>
+  <xacro:property name="proximal_link_mass" value="0.01"/>
+  <xacro:property name="distal_link_mass"   value="0.01"/>
+  <xacro:property name="proximal_pad_mass"  value="0.01"/>
+  <xacro:property name="distal_pad_mass"    value="0.01"/>
+  <xacro:property name="swivel_link_mass"   value="0.01"/>
+  <xacro:property name="base_link_mass"   value="0.74"/>
+  <xacro:property name="pad_mass"           value="0.1"/>
 <!-- ################ ################ ################ ################ ################ ################ -->
 <!-- ################ XACRO PORTION OF THE URDF, FOR MAKING THE FLEXIBLE JOINTS ################ -->
@@ -26,157 +38,4 @@
     <color rgba="0.2 0.8 0.75 1"/>
   </xacro:macro>
-  <!-- Macro to make each part of the link -->
-  <xacro:macro name="flex_link" params="finger_id flex_id">
-    <link
-      name="finger[${finger_id}]/flex_link[${flex_id}]">
-      <inertial>
-      <!-- TODO: CALCULATES CENTER OF MASS -->
-      <origin xyz="0.0 0.0 0.0"/>
-      <!-- TODO: CALCULATES THE MASS AND INERTIAs -->
-      <mass value="0.01"/>
-      <inertia
-        ixx="0.0001" ixy="0.0" ixz="0.0"
-                         iyy="0.0001"  iyz="0.0"
-                                           izz="0.0001"/>
-    </inertial>
-      <visual>
-        <origin
-          xyz="0 -0.008 0.001"
-          rpy="${pi/2} 0 ${pi/2}" />
-        <geometry>
-          <mesh
-            filename="package://reflex_description/meshes/flex_block.STL" />
-        </geometry>
-        <material
-          name="">
-          <xacro:flex_color/>
-        </material>
-      </visual>
-      <collision>
-      <origin xyz="0 -0.008 0.001" rpy="${pi/2} 0 ${pi/2}" />
-      <geometry>
-        <mesh filename="package://reflex_description/meshes/flex_block.STL" />
-      </geometry>
-    </collision>
-    </link>
-    <link name="finger[${finger_id}]/flex_link[${flex_id}]/virtual_link[1]"/>
-    <link name="finger[${finger_id}]/flex_link[${flex_id}]/virtual_link[2]"/>
-  </xacro:macro>
-  <!-- Macro to one flex body link to the next -->
-  <xacro:macro name="flex_joint" params="finger_id link_parent link_child">
-    <joint name="finger[${finger_id}]/flex_link[${link_parent}]/flex_joint_from_flex_link[${link_parent}]_to_virtual_link[1]" type="continuous">
-      <parent link="finger[${finger_id}]/flex_link[${link_parent}]"/>
-      <child link="finger[${finger_id}]/flex_link[${link_parent}]/virtual_link[1]"/>
-      <origin xyz="${flex_length/num_steps} 0 0" />
-      <axis xyz="0 -1 0"/>
-    </joint>
-    <joint name="finger[${finger_id}]/flex_link[${link_parent}]/flex_joint_from_virtual_link[1]_to_virtual_link[2]" type="continuous">
-      <parent link="finger[${finger_id}]/flex_link[${link_parent}]/virtual_link[1]"/>
-      <child link="finger[${finger_id}]/flex_link[${link_parent}]/virtual_link[2]"/>
-      <origin xyz="0 0 0" />
-      <axis xyz="-1 0 0"/>
-    </joint>
-    <joint name="finger[${finger_id}]/flex_link[${link_parent}]/flex_joint_from_virtual_link[2]_to_flex_link[${link_child}]" type="continuous">
-      <parent link="finger[${finger_id}]/flex_link[${link_parent}]/virtual_link[2]"/>
-      <child link="finger[${finger_id}]/flex_link[${link_child}]"/>
-      <origin xyz="0 0 0" />
-      <axis xyz="0 0 -1"/>
-    </joint>
-  </xacro:macro>
-  <!-- Macro to make the joint from proximal to first link and from last link to distal  -->
-  <xacro:macro name="flex_to_segment_joint" params="finger_id">
-    <link name="finger[${finger_id}]/prox/virtual_link[1]"/>
-    <link name="finger[${finger_id}]/prox/virtual_link[2]"/>
-    <joint name="finger[${finger_id}]/prox/flex_joint_from_prox_to_virtual_link[1]" type="continuous">
-      <parent link="proximal_${finger_id}"/>
-      <child link="finger[${finger_id}]/prox/virtual_link[1]"/>
-      <origin xyz="${prox_length} 0 -0.004"/>
-      <axis xyz="0 -1 0"/>
-    </joint>
-    <joint name="finger[${finger_id}]/prox/flex_joint_from_virtual_link[1]_to_virtual_link[2]" type="continuous">
-      <parent link="finger[${finger_id}]/prox/virtual_link[1]"/>
-      <child link="finger[${finger_id}]/prox/virtual_link[2]"/>
-      <origin xyz="0 0 0"/>
-      <axis xyz="-1 0 0"/>
-    </joint>
-    <joint name="finger[${finger_id}]/prox/flex_joint_from_virtual_link[2]_to_flex_link[1]" type="continuous">
-      <parent link="finger[${finger_id}]/prox/virtual_link[2]"/>
-      <child link="finger[${finger_id}]/flex_link[1]"/>
-      <origin xyz="0 0 0"/>
-      <axis xyz="0 0 -1"/>
-    </joint>
-    <joint name="finger[${finger_id}]/flex_link[${num_steps}]/flex_joint_from_flex_link[${num_steps}]_to_virtual_link[1]" type="continuous">
-      <parent link="finger[${finger_id}]/flex_link[${num_steps}]"/>
-      <child link="finger[${finger_id}]/flex_link[${num_steps}]/virtual_link[1]"/>
-      <origin xyz="${flex_length/num_steps-0.01} 0 0.008"/>
-      <axis xyz="0 -1 0"/>
-    </joint>
-    <joint name="finger[${finger_id}]/flex_link[${num_steps}]/flex_joint_from_virtual_link[1]_to_virtual_link[2]" type="continuous">
-      <parent link="finger[${finger_id}]/flex_link[${num_steps}]/virtual_link[1]"/>
-      <child link="finger[${finger_id}]/flex_link[${num_steps}]/virtual_link[2]"/>
-      <origin xyz="0 0 0"/>
-      <axis xyz="-1 0 0"/>
-    </joint>
-    <joint name="finger[${finger_id}]/flex_link[${num_steps}]/flex_joint_from_virtual_link[2]_to_dist" type="continuous">
-      <parent link="finger[${finger_id}]/flex_link[${num_steps}]/virtual_link[2]"/>
-      <child link="distal_${finger_id}"/>
-      <origin xyz="0 0 0"/>
-      <axis xyz="0 0 -1"/>
-    </joint>
-  </xacro:macro>
-  <xacro:flex_link finger_id="1" flex_id="1"/>
-  <xacro:flex_link finger_id="1" flex_id="2"/>
-  <xacro:flex_link finger_id="1" flex_id="3"/>
-  <xacro:flex_link finger_id="1" flex_id="4"/>
-  <xacro:flex_link finger_id="1" flex_id="5"/>
-  <xacro:flex_link finger_id="1" flex_id="6"/>
-  <xacro:flex_link finger_id="1" flex_id="7"/>
-  <xacro:flex_link finger_id="1" flex_id="8"/>
-  <xacro:flex_link finger_id="1" flex_id="9"/>
-  <xacro:flex_joint finger_id="1" link_parent="1" link_child="2"/>
-  <xacro:flex_joint finger_id="1" link_parent="2" link_child="3"/>
-  <xacro:flex_joint finger_id="1" link_parent="3" link_child="4"/>
-  <xacro:flex_joint finger_id="1" link_parent="4" link_child="5"/>
-  <xacro:flex_joint finger_id="1" link_parent="5" link_child="6"/>
-  <xacro:flex_joint finger_id="1" link_parent="6" link_child="7"/>
-  <xacro:flex_joint finger_id="1" link_parent="7" link_child="8"/>
-  <xacro:flex_joint finger_id="1" link_parent="8" link_child="9"/>
-  <xacro:flex_to_segment_joint finger_id="1"/>
-  <xacro:flex_link finger_id="2" flex_id="1"/>
-  <xacro:flex_link finger_id="2" flex_id="2"/>
-  <xacro:flex_link finger_id="2" flex_id="3"/>
-  <xacro:flex_link finger_id="2" flex_id="4"/>
-  <xacro:flex_link finger_id="2" flex_id="5"/>
-  <xacro:flex_link finger_id="2" flex_id="6"/>
-  <xacro:flex_link finger_id="2" flex_id="7"/>
-  <xacro:flex_link finger_id="2" flex_id="8"/>
-  <xacro:flex_link finger_id="2" flex_id="9"/>
-  <xacro:flex_joint finger_id="2" link_parent="1" link_child="2"/>
-  <xacro:flex_joint finger_id="2" link_parent="2" link_child="3"/>
-  <xacro:flex_joint finger_id="2" link_parent="3" link_child="4"/>
-  <xacro:flex_joint finger_id="2" link_parent="4" link_child="5"/>
-  <xacro:flex_joint finger_id="2" link_parent="5" link_child="6"/>
-  <xacro:flex_joint finger_id="2" link_parent="6" link_child="7"/>
-  <xacro:flex_joint finger_id="2" link_parent="7" link_child="8"/>
-  <xacro:flex_joint finger_id="2" link_parent="8" link_child="9"/>
-  <xacro:flex_to_segment_joint finger_id="2"/>
-  <xacro:flex_link finger_id="3" flex_id="1"/>
-  <xacro:flex_link finger_id="3" flex_id="2"/>
-  <xacro:flex_link finger_id="3" flex_id="3"/>
-  <xacro:flex_link finger_id="3" flex_id="4"/>
-  <xacro:flex_link finger_id="3" flex_id="5"/>
-  <xacro:flex_link finger_id="3" flex_id="6"/>
-  <xacro:flex_link finger_id="3" flex_id="7"/>
-  <xacro:flex_link finger_id="3" flex_id="8"/>
-  <xacro:flex_link finger_id="3" flex_id="9"/>
-  <xacro:flex_joint finger_id="3" link_parent="1" link_child="2"/>
-  <xacro:flex_joint finger_id="3" link_parent="2" link_child="3"/>
-  <xacro:flex_joint finger_id="3" link_parent="3" link_child="4"/>
-  <xacro:flex_joint finger_id="3" link_parent="4" link_child="5"/>
-  <xacro:flex_joint finger_id="3" link_parent="5" link_child="6"/>
-  <xacro:flex_joint finger_id="3" link_parent="6" link_child="7"/>
-  <xacro:flex_joint finger_id="3" link_parent="7" link_child="8"/>
-  <xacro:flex_joint finger_id="3" link_parent="8" link_child="9"/>
-  <xacro:flex_to_segment_joint finger_id="3"/>
 <!-- ################ ################ ################ ################ ################ ################ -->
 <!-- ################ THE SECTION CREATED BY SOLIDWORKS EXPORTER, CUT AND PASTE THIS IN HERE ################ -->
@@ -385,9 +244,9 @@
     </inertial>
     <visual>
-        <origin
-          xyz="0 -0.008 0.001" rpy="${pi/2} 0 ${pi/2}" />
+        <!-- <origin xyz="${flex_length/2.0} -0.008 0.001" rpy="${pi/2} 0 ${pi/2}" /> -->
+        <origin xyz="${flex_length/2.0} 0.0 0.0" rpy="0.0 0.0 0.0" />
         <geometry>
-          <mesh
-            filename="package://reflex_description/meshes/flex_block.STL" />
+          <!-- <mesh filename="package://reflex_description/meshes/flex_block.STL" /> -->
+          <box size="${flex_length*1.0} 0.014 0.006"/>
         </geometry>
         <material
@@ -397,7 +256,9 @@
       </visual>
     <collision>
-      <origin xyz="0 -0.008 0.001" rpy="${pi/2} 0 ${pi/2}" />
-      <geometry>
-        <mesh filename="package://reflex_description/meshes/flex_block.STL" />
+      <!-- <origin xyz="${flex_length/2.0} -0.008 0.001" rpy="${pi/2} 0 ${pi/2}" /> -->
+      <origin xyz="${flex_length/2.0} 0.0 0.0" rpy="0.0 0.0 0.0" />
+      <geometry>
+        <!-- <mesh filename="package://reflex_description/meshes/flex_block.STL" /> -->
+        <box size="${flex_length*1.0} 0.014 0.006"/>
       </geometry>
     </collision>
@@ -409,5 +270,5 @@
     <!-- <origin xyz="0.060 0 0.003"/>
     <axis xyz="0 -1 0"/> -->
-    <origin xyz="${flex_length} 0 0" />
+    <origin xyz="${prox_length} 0 ${0.001}" />
       <axis xyz="0 -1 0"/>
   </joint>
@@ -425,4 +286,5 @@
     <visual>
       <origin xyz="-0.077 0.007 0.007" rpy="3.1459 0 0" />
+      <!-- <origin xyz="0.0 0.0 0.0" rpy="3.1459 0 0" /> -->
       <geometry>
         <mesh
@@ -436,4 +298,5 @@
     <collision>
       <origin xyz="-0.077 0.007 0.007" rpy="3.1459 0 0" />
+      <!-- <origin xyz="0.0 0.0 0.0" rpy="3.1459 0 0" /> -->
       <geometry>
         <mesh filename="package://reflex_description/meshes/distal_1.STL" />
@@ -441,5 +304,6 @@
     </collision>
   </link>
-  <joint name="distal_joint_1" type="revolute">
+  <joint name="distal_joint_1"  type="continuous">
+    <!-- type="revolute"> -->
     <!-- type="continuous"> -->
     <!-- <origin
@@ -452,9 +316,12 @@
     <axis
       xyz="0 -1 0" /> -->
-    <origin xyz="0.0 0 0.003" rpy="0 0 0" />
+    <!-- <origin xyz="${flex_length} 0 0.00250000000000002" rpy="0 0 0" /> -->
+    <!-- <origin xyz="${flex_length-0.01} 0 0.008" rpy="0 0 0" /> -->
+    <!-- <origin xyz="${flex_length-0.01} 0 0.000" rpy="0 0 0" /> -->
+    <origin xyz="0.0 0 0.0" rpy="0 0 0" />
     <parent link="flex_link_1" />
     <child link="distal_1" />
     <axis xyz="0 -1 0" />
-    <limit effort="0.25" velocity="1.0" lower="0" upper="2.74" />
+    <!-- <limit effort="0.25" velocity="1.0" lower="0" upper="2.74" /> -->
   </joint>
   <link name="distal_pad_1">

Commit message: add the first part of finger 2, works

File: reflex_description/urdf/reflex_takktile_2.xacro (robot description, xacro)
@@ -117,4 +117,5 @@
       xyz="0 0 0" />
   </joint>
+  <!-- *****************************************FINGER 1**************************************************** -->
   <link name="swivel_1">
     <inertial>
@@ -362,4 +363,14 @@
   <!-- *****************************************FINGER 2**************************************************** -->
   <link name="swivel_2">
+    <inertial>
+      <!-- TODO: CALCULATES CENTER OF MASS -->
+      <origin xyz="0.0 0.0 0.0"/>
+      <!-- TODO: CALCULATES THE MASS AND INERTIAs -->
+      <mass value="0.01"/>
+      <inertia
+        ixx="0.0001" ixy="0.0" ixz="0.0"
+                         iyy="0.0001"  iyz="0.0"
+                                           izz="0.0001"/>
+    </inertial>
     <visual>
       <origin
@@ -375,4 +386,10 @@
       </material>
     </visual>
+    <collision>
+      <origin xyz="0.0 0.0 0.0" rpy="0 0 0" />
+      <geometry>
+        <mesh filename="package://reflex_description/meshes/swivel_2.STL" />
+      </geometry>
+    </collision>
   </link>
   <joint name="preshape_2" type="continuous">
@@ -388,8 +405,16 @@
   </joint>
   <link name="proximal_2">
-    <visual>
-      <origin
-        xyz="-0.011 0.007 0.011"
-        rpy="3.1459 0 0"/>
+    <inertial>
+      <!-- TODO: CALCULATES CENTER OF MASS -->
+      <origin xyz="0.0 0.0 0.0"/>
+      <!-- TODO: CALCULATES THE MASS AND INERTIAs -->
+      <mass value="0.01"/>
+      <inertia
+        ixx="0.0001" ixy="0.0" ixz="0.0"
+                         iyy="0.0001"  iyz="0.0"
+                                           izz="0.0001"/>
+    </inertial>
+    <visual>
+      <origin xyz="-0.011 0.007 0.011" rpy="3.1459 0 0"/>
       <geometry>
         <mesh
@@ -401,4 +426,10 @@
       </material>
     </visual>
+    <collision>
+      <origin xyz="-0.011 0.007 0.011" rpy="3.1459 0 0"/>
+      <geometry>
+        <mesh filename="package://reflex_description/meshes/proximal_1.STL" />
+      </geometry>
+    </collision>
   </link>
   <joint name="proximal_joint_2" type="continuous">
@@ -414,8 +445,16 @@
   </joint>
   <link name="proximal_pad_2">
-    <visual>
-      <origin
-        xyz="-0.008 0.014 -0.002"
-        rpy="1.5708 1.5708 0" />
+    <inertial>
+      <!-- TODO: CALCULATES CENTER OF MASS -->
+      <origin xyz="0.0 0.0 0.0"/>
+      <!-- TODO: CALCULATES THE MASS AND INERTIAs -->
+      <mass value="0.01"/>
+      <inertia
+        ixx="0.0001" ixy="0.0" ixz="0.0"
+                         iyy="0.0001"  iyz="0.0"
+                                           izz="0.0001"/>
+    </inertial>
+    <visual>
+      <origin xyz="-0.008 0.014 -0.002" rpy="1.5708 1.5708 0" />
       <geometry>
         <mesh
@@ -427,4 +466,10 @@
       </material>
     </visual>
+    <collision>
+      <origin xyz="-0.008 0.014 -0.002" rpy="1.5708 1.5708 0" />
+      <geometry>
+        <mesh filename="package://reflex_description/meshes/proximal_pad_1.STL" />
+      </geometry>
+    </collision>
   </link>
   <joint name="prox2_pad_joint" type="fixed">
