Commit message: full hand add

File: reflex_description/urdf/reflex_takktile_2.xacro (robot description, xacro)
@@ -484,9 +484,56 @@
       xyz="0 0 0" />
   </joint>
+  <link name="flex_link_2">
+     <inertial>
+      <!-- TODO: CALCULATES CENTER OF MASS -->
+      <origin xyz="0.0 0.0 0.0"/>
+      <!-- TODO: CALCULATES THE MASS AND INERTIAs -->
+      <mass value="0.01"/>
+      <inertia
+        ixx="0.0001"  ixy="0.0"     ixz="0.0"
+                      iyy="0.0001"  iyz="0.0"
+                                    izz="0.0001"/>
+    </inertial>
+    <visual>
+        <origin xyz="${flex_length/2.0} 0.0 0.0" rpy="0.0 0.0 0.0" />
+        <geometry>
+          <!-- <mesh filename="package://reflex_description/meshes/flex_block.STL" /> -->
+          <box size="${flex_length*1.0} 0.014 0.006"/>
+        </geometry>
+        <material
+          name="">
+          <xacro:flex_color/>
+        </material>
+      </visual>
+    <collision>
+      <origin xyz="${flex_length/2.0} 0.0 0.0" rpy="0.0 0.0 0.0" />
+      <geometry>
+        <!-- <mesh filename="package://reflex_description/meshes/flex_block.STL" /> -->
+        <box size="${flex_length*1.0} 0.014 0.006"/>
+      </geometry>
+    </collision>
+  </link>
+  <!-- TODO: DISTANCE TO CHECK!!!! -->
+  <joint name="flex_joint_2" type="fixed">
+    <parent link="proximal_2"/>
+    <child link="flex_link_2"/>
+    <!-- <origin xyz="0.060 0 0.003"/>
+    <axis xyz="0 -1 0"/> -->
+    <origin xyz="${prox_length} 0 ${0.001}" />
+      <axis xyz="0 -1 0"/>
+  </joint>
   <link name="distal_2">
-    <visual>
-      <origin
-        xyz="-0.077 0.007 0.006"
-        rpy="3.1459 0 0" />
+    <inertial>
+      <!-- TODO: CALCULATES CENTER OF MASS -->
+      <origin xyz="0.0 0.0 0.0"/>
+      <!-- TODO: CALCULATES THE MASS AND INERTIAs -->
+      <mass value="0.01"/>
+      <inertia
+        ixx="0.0001"  ixy="0.0"     ixz="0.0"
+                      iyy="0.0001"  iyz="0.0"
+                                    izz="0.0001"/>
+    </inertial>
+    <visual>
+      <origin xyz="-0.077 0.007 0.006" rpy="3.1459 0 0" />
       <geometry>
         <mesh
@@ -498,11 +545,16 @@
       </material>
     </visual>
+    <collision>
+      <origin xyz="-0.077 0.007 0.006" rpy="3.1459 0 0" />
+      <geometry>
+        <mesh filename="package://reflex_description/meshes/distal_1.STL" />
+        <!-- <box size="${flex_length*1.0} 0.014 0.006"/> -->
+      </geometry>
+    </collision>
   </link>
   <joint name="distal_joint_2" type="continuous">
-    <origin
-      xyz="0.0760000000000001 0 0.00249999999999997"
-      rpy="0 0 0" />
-    <parent
-      link="proximal_2" />
+    <origin xyz="${flex_length-0.01} 0 0.001" rpy="0 0 0" />
+    <parent
+      link="flex_link_2" />
     <child
       link="distal_2" />
@@ -511,11 +563,18 @@
   </joint>
   <link name="distal_pad_2">
-    <visual>
-      <origin
-        xyz="-0.00825 0.009 0.057"
-        rpy="1.5708 1.5708 0" />
-      <geometry>
-        <mesh
-          filename="package://reflex_description/meshes/distal_pad_1.STL" />
+    <inertial>
+      <!-- TODO: CALCULATES CENTER OF MASS -->
+      <origin xyz="0.0 0.0 0.0"/>
+      <!-- TODO: CALCULATES THE MASS AND INERTIAs -->
+      <mass value="0.01"/>
+      <inertia
+        ixx="0.0001"  ixy="0.0"     ixz="0.0"
+                      iyy="0.0001"  iyz="0.0"
+                                    izz="0.0001"/>
+    </inertial>
+    <visual>
+      <origin xyz="-0.00825 0.009 0.057" rpy="1.5708 1.5708 0" />
+      <geometry>
+        <mesh filename="package://reflex_description/meshes/distal_pad_1.STL" />
       </geometry>
       <material
@@ -524,4 +583,10 @@
       </material>
     </visual>
+    <collision>
+      <origin xyz="-0.00825 0.009 0.057" rpy="1.5708 1.5708 0" />
+      <geometry>
+        <mesh filename="package://reflex_description/meshes/distal_pad_1.STL" />
+      </geometry>
+    </collision>
   </link>
   <joint name="dist2_pad_joint" type="fixed">
@@ -536,9 +601,18 @@
       xyz="0 0 0" />
   </joint>
+<!-- *****************************************FINGER 3**************************************************** -->
   <link name="proximal_3">
-    <visual>
-      <origin
-        xyz="-0.011 0.007 0.011"
-        rpy="3.1459 0 0"/>
+    <inertial>
+      <!-- TODO: CALCULATES CENTER OF MASS -->
+      <origin xyz="0.0 0.0 0.0"/>
+      <!-- TODO: CALCULATES THE MASS AND INERTIAs -->
+      <mass value="0.01"/>
+      <inertia
+        ixx="0.0001" ixy="0.0" ixz="0.0"
+                         iyy="0.0001"  iyz="0.0"
+                                           izz="0.0001"/>
+    </inertial>
+    <visual>
+      <origin xyz="-0.011 0.007 0.011" rpy="3.1459 0 0"/>
       <geometry>
         <mesh
@@ -550,6 +624,11 @@
       </material>
     </visual>
-  </link>
-<!-- *****************************************FINGER 3**************************************************** -->
+    <collision>
+      <origin xyz="-0.011 0.007 0.011" rpy="3.1459 0 0"/>
+      <geometry>
+        <mesh filename="package://reflex_description/meshes/proximal_1.STL" />
+      </geometry>
+    </collision>
+  </link>
   <joint name="proximal_joint_3" type="continuous">
     <origin
@@ -564,8 +643,16 @@
   </joint>
   <link name="proximal_pad_3">
-    <visual>
-      <origin
-        xyz="-0.008 0.014 -0.002"
-        rpy="1.5708 1.5708 0" />
+    <inertial>
+      <!-- TODO: CALCULATES CENTER OF MASS -->
+      <origin xyz="0.0 0.0 0.0"/>
+      <!-- TODO: CALCULATES THE MASS AND INERTIAs -->
+      <mass value="0.01"/>
+      <inertia
+        ixx="0.0001" ixy="0.0" ixz="0.0"
+                         iyy="0.0001"  iyz="0.0"
+                                           izz="0.0001"/>
+    </inertial>
+    <visual>
+      <origin xyz="-0.008 0.014 -0.002" rpy="1.5708 1.5708 0" />
       <geometry>
         <mesh
@@ -577,4 +664,10 @@
       </material>
     </visual>
+    <collision>
+      <origin xyz="-0.008 0.014 -0.002" rpy="1.5708 1.5708 0" />
+      <geometry>
+        <mesh filename="package://reflex_description/meshes/proximal_pad_1.STL" />
+      </geometry>
+    </collision>
   </link>
   <joint name="prox3_pad_joint" type="fixed">
@@ -589,9 +682,56 @@
       xyz="0 0 0" />
   </joint>
+  <link name="flex_link_3">
+     <inertial>
+      <!-- TODO: CALCULATES CENTER OF MASS -->
+      <origin xyz="0.0 0.0 0.0"/>
+      <!-- TODO: CALCULATES THE MASS AND INERTIAs -->
+      <mass value="0.01"/>
+      <inertia
+        ixx="0.0001"  ixy="0.0"     ixz="0.0"
+                      iyy="0.0001"  iyz="0.0"
+                                    izz="0.0001"/>
+    </inertial>
+    <visual>
+        <origin xyz="${flex_length/2.0} 0.0 0.0" rpy="0.0 0.0 0.0" />
+        <geometry>
+          <!-- <mesh filename="package://reflex_description/meshes/flex_block.STL" /> -->
+          <box size="${flex_length*1.0} 0.014 0.006"/>
+        </geometry>
+        <material
+          name="">
+          <xacro:flex_color/>
+        </material>
+      </visual>
+    <collision>
+      <origin xyz="${flex_length/2.0} 0.0 0.0" rpy="0.0 0.0 0.0" />
+      <geometry>
+        <!-- <mesh filename="package://reflex_description/meshes/flex_block.STL" /> -->
+        <box size="${flex_length*1.0} 0.014 0.006"/>
+      </geometry>
+    </collision>
+  </link>
+  <!-- TODO: DISTANCE TO CHECK!!!! -->
+  <joint name="flex_joint_3" type="fixed">
+    <parent link="proximal_3"/>
+    <child link="flex_link_3"/>
+    <!-- <origin xyz="0.060 0 0.003"/>
+    <axis xyz="0 -1 0"/> -->
+    <origin xyz="${prox_length} 0 ${0.001}" />
+      <axis xyz="0 -1 0"/>
+  </joint>
   <link name="distal_3">
-    <visual>
-      <origin
-        xyz="-0.077 0.007 0.006"
-        rpy="3.1459 0 0" />
+    <inertial>
+      <!-- TODO: CALCULATES CENTER OF MASS -->
+      <origin xyz="0.0 0.0 0.0"/>
+      <!-- TODO: CALCULATES THE MASS AND INERTIAs -->
+      <mass value="0.01"/>
+      <inertia
+        ixx="0.0001"  ixy="0.0"     ixz="0.0"
+                      iyy="0.0001"  iyz="0.0"
+                                    izz="0.0001"/>
+    </inertial>
+    <visual>
+      <origin xyz="-0.077 0.007 0.006" rpy="3.1459 0 0" />
       <geometry>
         <mesh
@@ -603,11 +743,15 @@
       </material>
     </visual>
+    <collision>
+      <origin xyz="-0.077 0.007 0.006" rpy="3.1459 0 0" />
+      <geometry>
+        <mesh filename="package://reflex_description/meshes/distal_1.STL" />
+      </geometry>
+    </collision>
   </link>
   <joint name="distal_joint_3" type="continuous">
-    <origin
-      xyz="0.0760000000000001 0 0.0025"
-      rpy="-1.48887961834512E-45 -1.0995850059156E-76 -7.38531841236285E-32" />
-    <parent
-      link="proximal_3" />
+    <origin xyz="${flex_length-0.01} 0 0.001" rpy="0 0 0" />
+    <parent
+      link="flex_link_3" />
     <child
       link="distal_3" />
@@ -616,8 +760,16 @@
   </joint>
   <link name="distal_pad_3">
-    <visual>
-      <origin
-        xyz="-0.00825 0.009 0.057"
-        rpy="1.5708 1.5708 0" />
+    <inertial>
+      <!-- TODO: CALCULATES CENTER OF MASS -->
+      <origin xyz="0.0 0.0 0.0"/>
+      <!-- TODO: CALCULATES THE MASS AND INERTIAs -->
+      <mass value="0.01"/>
+      <inertia
+        ixx="0.0001"  ixy="0.0"     ixz="0.0"
+                      iyy="0.0001"  iyz="0.0"
+                                    izz="0.0001"/>
+    </inertial>
+    <visual>
+      <origin xyz="-0.00825 0.009 0.057" rpy="1.5708 1.5708 0" />
       <geometry>
         <mesh
@@ -629,4 +781,10 @@
       </material>
     </visual>
+    <collision>
+      <origin xyz="-0.00825 0.009 0.057" rpy="1.5708 1.5708 0" />
+      <geometry>
+        <mesh filename="package://reflex_description/meshes/distal_pad_1.STL" />
+      </geometry>
+    </collision>
   </link>
   <joint name="dist3_pad_joint" type="fixed">

Commit message: add the limit of the joints

File: reflex_description/urdf/reflex_takktile_2.xacro (robot description, xacro)
@@ -14,6 +14,17 @@
   <xacro:property name="distal_pad_mass"    value="0.01"/>
   <xacro:property name="swivel_link_mass"   value="0.01"/>
-  <xacro:property name="base_link_mass"   value="0.74"/>
+  <xacro:property name="base_link_mass"     value="0.74"/>
   <xacro:property name="pad_mass"           value="0.1"/>
+<!-- Parameters joints -->
+  <!-- Preshape -->
+  <xacro:property name="preshape_joint_limit_lower"      value="-0.0872665"/>
+  <xacro:property name="preshape_joint_limit_upper"      value="2.09440"/>
+  <xacro:property name="preshape_joint_limit_velocity"   value="1.0"/>
+  <xacro:property name="preshape_joint_limit_effort"     value="30.0"/>
+  <!-- Proximal -->
+  <xacro:property name="proximal_joint_limit_lower"      value="0.0"/>
+  <xacro:property name="proximal_joint_limit_upper"      value="2.09440"/>
+  <xacro:property name="proximal_joint_limit_velocity"   value="1.0"/>
+  <xacro:property name="proximal_joint_limit_effort"     value="30.0"/>
 <!-- ################ ################ ################ ################ ################ ################ -->
 <!-- ################ XACRO PORTION OF THE URDF, FOR MAKING THE FLEXIBLE JOINTS ################ -->
@@ -130,14 +141,16 @@
     </collision>
   </link>
-  <joint name="preshape_1" type="continuous">
+  <joint name="preshape_1" type="revolute">
     <origin
       xyz="0.0503973683071414 -0.026 0.063"
       rpy="6.75550818663469E-16 1.97993848419069E-16 -2.77555756156289E-16" />
-    <parent
-      link="base_link" />
-    <child
-      link="swivel_1" />
-    <axis
-      xyz="0 0 -1" />
+    <parent link="base_link" />
+    <child link="swivel_1" />
+    <axis xyz="0 0 -1" />
+    <!-- <limit effort="30" velocity="1.0" lower="-0.0872665" upper="2.0944" /> -->
+    <limit effort="${preshape_joint_limit_effort}"
+            velocity="${preshape_joint_limit_velocity}"
+            lower="${preshape_joint_limit_lower}"
+            upper="${preshape_joint_limit_upper}" />
   </joint>
   <link name="proximal_1">
@@ -170,14 +183,15 @@
     </collision>
   </link>
-  <joint name="proximal_joint_1" type="continuous">
+  <joint name="proximal_joint_1" type="revolute">
     <origin
       xyz="0.01 0 0.0186"
       rpy="-6.20039667432211E-16 0.05 2.22044604925031E-16" />
-    <parent
-      link="swivel_1" />
-    <child
-      link="proximal_1" />
-    <axis
-      xyz="0 -1 0" />
+    <parent link="swivel_1" />
+    <child link="proximal_1" />
+    <axis xyz="0 -1 0" />
+    <limit effort="${proximal_joint_limit_effort}"
+            velocity="${proximal_joint_limit_velocity}"
+            lower="${proximal_joint_limit_lower}"
+            upper="${proximal_joint_limit_upper}" />
   </joint>
   <link name="proximal_pad_1">
@@ -376,14 +390,16 @@
     </collision>
   </link>
-  <joint name="preshape_2" type="continuous">
+  <joint name="preshape_2" type="revolute">
     <origin
       xyz="0.0503973683071413 0.0259999999999999 0.063"
       rpy="1.22459340959228E-15 -7.33448407631817E-16 -1.66533453693773E-16" />
-    <parent
-      link="base_link" />
-    <child
-      link="swivel_2" />
-    <axis
-      xyz="0 0 -1" />
+    <parent link="base_link" />
+    <child link="swivel_2" />
+    <axis xyz="0 0 -1" />
+    <!-- <limit effort="30" velocity="1.0" lower="-0.0872665" upper="2.0944" /> -->
+    <limit effort="${preshape_joint_limit_effort}"
+            velocity="${preshape_joint_limit_velocity}"
+            lower="${preshape_joint_limit_lower}"
+            upper="${preshape_joint_limit_upper}" />
   </joint>
   <link name="proximal_2">
@@ -416,14 +432,15 @@
     </collision>
   </link>
-  <joint name="proximal_joint_2" type="continuous">
+  <joint name="proximal_joint_2" type="revolute">
     <origin
       xyz="0.01 0 0.0186"
       rpy="-1.16908225836102E-15 0.05 1.11022302462515E-16" />
-    <parent
-      link="swivel_2" />
-    <child
-      link="proximal_2" />
-    <axis
-      xyz="0 -1 0" />
+    <parent link="swivel_2" />
+    <child link="proximal_2" />
+    <axis xyz="0 -1 0" />
+    <limit effort="${proximal_joint_limit_effort}"
+            velocity="${proximal_joint_limit_velocity}"
+            lower="${proximal_joint_limit_lower}"
+            upper="${proximal_joint_limit_upper}" />
   </joint>
   <link name="proximal_pad_2">
@@ -614,14 +631,15 @@
     </collision>
   </link>
-  <joint name="proximal_joint_3" type="continuous">
+  <joint name="proximal_joint_3" type="revolute">
     <origin
       xyz="-0.0299999999999996 0 0.0816000000000002"
       rpy="-5.55111512312578E-17 0.05 3.14159265358979" />
-    <parent
-      link="base_link" />
-    <child
-      link="proximal_3" />
-    <axis
-      xyz="0 -1 0" />
+    <parent link="base_link" />
+    <child link="proximal_3" />
+    <axis xyz="0 -1 0" />
+    <limit effort="${proximal_joint_limit_effort}"
+            velocity="${proximal_joint_limit_velocity}"
+            lower="${proximal_joint_limit_lower}"
+            upper="${proximal_joint_limit_upper}" />
   </joint>
   <link name="proximal_pad_3">

Commit message: before add a mass to end effector

File: reflex_description/urdf/reflex_takktile_2.xacro (robot description, xacro)
@@ -12,4 +12,6 @@
   <xacro:include filename="$(find reflex_description)/materials/reflex.materials.xacro" />
   <xacro:include filename="$(find reflex_description)/urdf/tactile_sensors.xacro" />
+  <xacro:include filename="$(find iiwa_description)/urdf/iiwa7.xacro"/>
+  <xacro:include filename="$(find iiwa_description)/urdf/iiwa7.urdf.xacro"/>
 <!-- Properties -->
   <xacro:property name="flex_link_mass"     value="0.01"/>
@@ -83,9 +85,9 @@
   </link>
   <!-- For a tool on a arm, uncomment this part -->
-  <!-- <joint name="tool_joint" type="fixed">
+  <joint name="tool_joint" type="fixed">
       <parent link="iiwa_link_ee" />
       <child link = "base_link" />
       <origin xyz="0.0 0.0 0.0" rpy="0 0.0 3.14159" />
-  </joint> -->
+  </joint>
   <link name="pad">
     <inertial>
@@ -128,4 +130,13 @@
       xyz="0 0 0" />
   </joint>
+  <!-- Add the tool tips which is the pose of the hand effector -->
+  <!-- TODO Check the offset of the tool! -->
+  <joint name="tool_ee_joint" type="fixed">
+  <parent link="base_link" />
+  <child link = "tool_link_ee" />
+  <origin xyz="0 0 0.1275" rpy="0 ${0.0/1.0} 0" />
+</joint>
+<!--  The TCP frame is here defined -->
+<link name="tool_link_ee"/>
 <!-- *****************************************FINGER 1**************************************************** -->
   <link name="swivel_1">

Commit message: add travis for trying

File: reflex_description/urdf/reflex_takktile_2.xacro (robot description, xacro)
@@ -138,5 +138,32 @@
 </joint>
 <!--  The TCP frame is here defined -->
-<link name="tool_link_ee"/>
+<link name="tool_link_ee">
+  <inertial>
+    <!-- TODO: CALCULATES CENTER OF MASS -->
+    <origin xyz="0.0 0.0 0.0"/>
+    <!-- TODO: CALCULATES THE MASS AND INERTIAs -->
+    <mass value="0.0001"/>
+    <inertia
+      ixx="0.0001" ixy="0.0" ixz="0.0"
+                        iyy="0.0001"  iyz="0.0"
+                                          izz="0.0001"/>
+  </inertial>
+  <visual>
+    <origin xyz="0 0 0" rpy="0 0 0" />
+    <geometry>
+     <cylinder length="${length}" radius="${radius}"/>
+    </geometry>
+    <material
+      name="">
+      <xacro:pad_color/>
+    </material>
+  </visual>
+  <collision>
+    <origin xyz="0.0 0.0 0.0" rpy="0 0 0" />
+    <geometry>
+      <cylinder length="${length}" radius="${radius}"/>
+    </geometry>
+  </collision>
+</link>
 <!-- *****************************************FINGER 1**************************************************** -->
   <link name="swivel_1">

Commit message: small modification for rl part

File: reflex_description/urdf/reflex_takktile_2.xacro (robot description, xacro)
@@ -139,8 +139,6 @@
 <!--  The TCP frame is here defined -->
 <link name="tool_link_ee">
-  <inertial>
-    <!-- TODO: CALCULATES CENTER OF MASS -->
+  <!-- <inertial>
     <origin xyz="0.0 0.0 0.0"/>
-    <!-- TODO: CALCULATES THE MASS AND INERTIAs -->
     <mass value="0.0001"/>
     <inertia
@@ -164,5 +162,5 @@
       <cylinder length="${length}" radius="${radius}"/>
     </geometry>
-  </collision>
+  </collision> -->
 </link>
 <!-- *****************************************FINGER 1**************************************************** -->

Commit message: add the plate to have a ground

File: reflex_description/urdf/reflex_takktile_2.xacro (robot description, xacro)
@@ -738,4 +738,35 @@
     <axis xyz="0 0 0" />
   </joint>
+  <!-- Create flat square under the robot -->
+  <!-- <box size="0.19 0.19 0.07"/> -->
+  <link name="ground">
+    <inertial>
+      <origin xyz="0.0 0.0 0.0"/>
+      <mass value="100000"/>
+      <inertia ixx="100000" ixy="0.0" ixz="0.0" iyy="100000.0001" iyz="0.0" izz="100000.0001"/>
+    </inertial>
+    <visual>
+      <origin xyz="0 0 0" rpy="0 0 0" />
+      <geometry>
+        <box size="2.0 2. 0.0001"/>
+      </geometry>
+      <!-- <material name="base_color">
+        <xacro:base_color/>
+      </material> -->
+    </visual>
+    <!-- TODO: Change the BASE OF the hand to the version 2 -->
+    <collision>
+      <origin xyz="0.0 0.0 0.0" rpy="0 0 0" />
+      <geometry>
+        <box size="2.0 2. 0.0001"/>
+      </geometry>
+    </collision>
+  </link>
+  <!-- For a tool on a arm, uncomment this part -->
+  <joint name="ground_link" type="fixed">
+    <parent link="iiwa_link_0" />
+    <child link = "ground" />
+    <origin xyz="0.0 0.0 0.0" rpy="0 0.0 3.14159" />
+  </joint>
   <!-- ******************************************************************************************************* -->
   <!-- Objects to drop -->
