Commit message: add an urdf

File: reflex_description/urdf/object_to_catch.urdf (robot description, URDF)
Before this commit: robot object_to_catch, 1 links, 0 joints
Links:
- link link: mass ${mass} -> 0.8; geometry collision box size=0.06 0.3 0.08; visual box size=0.06 0.3 0.08

File: reflex_description/urdf/reflex_takktile_2.xacro (robot description, xacro)
@@ -16,12 +16,12 @@
   <xacro:include filename="$(find iiwa_description)/urdf/iiwa7.urdf.xacro"/>
   <!-- Properties -->
-  <xacro:property name="flex_link_mass" value="0.01"/>
-  <xacro:property name="proximal_link_mass" value="0.01"/>
-  <xacro:property name="distal_link_mass" value="0.01"/>
-  <xacro:property name="proximal_pad_mass" value="0.01"/>
-  <xacro:property name="distal_pad_mass" value="0.01"/>
-  <xacro:property name="swivel_link_mass" value="0.01"/>
-  <xacro:property name="base_link_mass" value="0.34"/><!-- 0.74 -->
-  <xacro:property name="pad_mass" value="0.1"/>
+  <xacro:property name="flex_link_mass" value="0.0001"/>
+  <xacro:property name="proximal_link_mass" value="0.0001"/>
+  <xacro:property name="distal_link_mass" value="0.0001"/>
+  <xacro:property name="proximal_pad_mass" value="0.0001"/>
+  <xacro:property name="distal_pad_mass" value="0.0001"/>
+  <xacro:property name="swivel_link_mass" value="0.0001"/>
+  <xacro:property name="base_link_mass" value="0.0074"/><!-- 0.74 -->
+  <xacro:property name="pad_mass" value="0.001"/>
   <!-- Parameters Limits Joints -->
   <!-- Preshape -->

Commit message: modify parameter for grip

File: reflex_description/urdf/object_to_catch.urdf (robot description, URDF)
Before this commit: robot object_to_catch, 1 links, 0 joints
Links:
- link link: geometry collision box size=0.14 0.3 0.08; visual box size=0.14 0.3 0.08

File: reflex_description/urdf/reflex.gazebo.xacro (robot description, xacro)
@@ -191,8 +191,8 @@
       <forces_angle_tolerance>90</forces_angle_tolerance>
       <update_rate>100</update_rate>
-      <grip_count_threshold>6</grip_count_threshold>
+      <grip_count_threshold>3</grip_count_threshold>
       <max_grip_count>20</max_grip_count>
-      <release_tolerance>0.05</release_tolerance>
-      <disable_collisions_on_attach>true</disable_collisions_on_attach>
+      <release_tolerance>0.09</release_tolerance>
+      <disable_collisions_on_attach>false</disable_collisions_on_attach>
       <contact_topic>__default_topic__</contact_topic>
     </plugin>

Commit message: up

File: reflex_description/urdf/object_to_catch.urdf (robot description, URDF)
Before this commit: robot object_to_catch, 1 links, 0 joints
Links:
- link link: geometry collision box size=0.20 0.20 0.08; visual box size=0.20 0.20 0.08

File: reflex_description/urdf/object_to_catch.xacro (robot description, xacro)
@@ -15,6 +15,6 @@
   <xacro:include filename="$(find iiwa_description)/urdf/iiwa7.urdf.xacro"/> -->
 <!-- Properties -->
-  <xacro:property name="rectangle_x"     value="0.06"/>
-  <xacro:property name="rectangle_y" value="0.300"/>
+  <xacro:property name="rectangle_x"     value="0.20"/>
+  <xacro:property name="rectangle_y" value="0.20"/>
   <xacro:property name="rectangle_z"   value="0.08"/>
   <xacro:property name="mass"   value="0.80"/>
@@ -34,12 +34,4 @@
                          iyy="${I_yy}"  iyz="0.0"
                                            izz="${I_zz}"/>
-        <!-- <inertia
-        ixx="0.1" ixy="0.0" ixz="0.0"
-                         iyy="0.1"  iyz="0.0"
-                                           izz="0.1"/> -->
-        <!-- <inertia
-        ixx="${0.083333 * mass * (rectangle_y*rectangle_y + rectangle_z*rectangle_z)}" ixy="0.0" ixz="0.0"
-                         iyy="${0.083333 * mass * (rectangle_x*rectangle_x + rectangle_z*rectangle_z)}"  iyz="0.0"
-                                           izz="{0.083333 * mass * (rectangle_y*rectangle_y + rectangle_x*rectangle_x)}"/> -->
     </inertial>
     <visual>

File: reflex_description/urdf/reflex.gazebo.xacro (robot description, xacro)
@@ -107,47 +107,4 @@
 			<!-- <maxContacts>1</maxContacts> -->
   </gazebo>
-  <!-- Add gazebo - pkg for grasping -->
-  <!-- <gazebo>
-   <plugin name="gazebo_grasp_fix" filename="libgazebo_grasp_fix.so">
-        <arm>
-           <arm_name>base_link</arm_name>
-           <palm_link>pad</palm_link>
-           <gripper_link>distal_pad_1</gripper_link>
-           <gripper_link>distal_pad_2</gripper_link>
-           <gripper_link>distal_pad_3</gripper_link>
-           <gripper_link>proximal_pad_1</gripper_link>
-           <gripper_link>proximal_pad_2</gripper_link>
-           <gripper_link>proximal_pad_3</gripper_link>
-        </arm>
-       <forces_angle_tolerance>100</forces_angle_tolerance>
-       <update_rate>4</update_rate>
-       <grip_count_threshold>4</grip_count_threshold>
-       <max_grip_count>8</max_grip_count>
-       <release_tolerance>0.005</release_tolerance>
-       <disable_collisions_on_attach>false</disable_collisions_on_attach>
-       <contact_topic>__default_topic__</contact_topic>
-    </plugin>
-  </gazebo> -->
-  <!-- <gazebo>
-   <plugin name="gazebo_grasp_fix" filename="libgazebo_grasp_fix.so">
-        <arm>
-           <arm_name>base_link</arm_name>
-           <palm_link>pad</palm_link>
-           <gripper_link>iiwa/distal_pad_1</gripper_link>
-           <gripper_link>iiwa/distal_pad_2</gripper_link>
-           <gripper_link>iiwa/distal_pad_3</gripper_link>
-           <gripper_link>iiwa/proximal_pad_1</gripper_link>
-           <gripper_link>iiwa/proximal_pad_2</gripper_link>
-           <gripper_link>iiwa/proximal_pad_3</gripper_link>
-        </arm>
-       <forces_angle_tolerance>100</forces_angle_tolerance>
-       <update_rate>10</update_rate>
-       <grip_count_threshold>2</grip_count_threshold>
-       <max_grip_count>10</max_grip_count>
-       <release_tolerance>0.005</release_tolerance>
-       <disable_collisions_on_attach>true</disable_collisions_on_attach>
-       <contact_topic>__default_topic__</contact_topic>
-    </plugin>
-  </gazebo> -->
   <gazebo>
    <plugin name="gazebo_grasp_fix" filename="libgazebo_grasp_fix.so">
@@ -198,51 +155,3 @@
     </plugin>
   </gazebo>
-  <!-- <gazebo>
-   <plugin name="gazebo_grasp_fix" filename="libgazebo_grasp_fix.so">
-        <arm>
-          <arm_name>base_link</arm_name>
-          <palm_link>iiwa/pad</palm_link>
-          <gripper_link>iiwa/distal_1</gripper_link>
-          <gripper_link>iiwa/distal_2</gripper_link>
-          <gripper_link>iiwa/distal_3</gripper_link>
-          <gripper_link>iiwa/proximal_1</gripper_link>
-          <gripper_link>iiwa/proximal_2</gripper_link>
-          <gripper_link>iiwa/proximal_3</gripper_link>
-          <gripper_link>iiwa/proximal_1_sensor_1</gripper_link>
-          <gripper_link>iiwa/proximal_1_sensor_2</gripper_link>
-          <gripper_link>iiwa/proximal_1_sensor_3</gripper_link>
-          <gripper_link>iiwa/proximal_1_sensor_4</gripper_link>
-          <gripper_link>iiwa/proximal_1_sensor_5</gripper_link>
-          <gripper_link>iiwa/proximal_2_sensor_1</gripper_link>
-          <gripper_link>iiwa/proximal_2_sensor_2</gripper_link>
-          <gripper_link>iiwa/proximal_2_sensor_3</gripper_link>
-          <gripper_link>iiwa/proximal_2_sensor_4</gripper_link>
-          <gripper_link>iiwa/proximal_2_sensor_5</gripper_link>
-          <gripper_link>iiwa/proximal_3_sensor_1</gripper_link>
-          <gripper_link>iiwa/proximal_3_sensor_2</gripper_link>
-          <gripper_link>iiwa/proximal_3_sensor_3</gripper_link>
-          <gripper_link>iiwa/proximal_3_sensor_4</gripper_link>
-          <gripper_link>iiwa/proximal_3_sensor_5</gripper_link>
-          <gripper_link>iiwa/distal_1_sensor_1</gripper_link>
-          <gripper_link>iiwa/distal_1_sensor_2</gripper_link>
-          <gripper_link>iiwa/distal_1_sensor_3</gripper_link>
-          <gripper_link>iiwa/distal_1_sensor_4</gripper_link>
-          <gripper_link>iiwa/distal_2_sensor_1</gripper_link>
-          <gripper_link>iiwa/distal_2_sensor_2</gripper_link>
-          <gripper_link>iiwa/distal_2_sensor_3</gripper_link>
-          <gripper_link>iiwa/distal_2_sensor_4</gripper_link>
-          <gripper_link>iiwa/distal_3_sensor_1</gripper_link>
-          <gripper_link>iiwa/distal_3_sensor_2</gripper_link>
-          <gripper_link>iiwa/distal_3_sensor_3</gripper_link>
-          <gripper_link>iiwa/distal_3_sensor_4</gripper_link>
-        </arm>
-      <forces_angle_tolerance>180</forces_angle_tolerance>
-      <update_rate>100</update_rate>
-      <grip_count_threshold>2</grip_count_threshold>
-      <max_grip_count>10</max_grip_count>
-      <release_tolerance>0.05</release_tolerance>
-      <disable_collisions_on_attach>true</disable_collisions_on_attach>
-      <contact_topic>__default_topic__</contact_topic>
-    </plugin>
-  </gazebo> -->
 </robot>

File: reflex_description/urdf/reflex_takktile_2.xacro (robot description, xacro)
@@ -16,26 +16,26 @@
   <xacro:include filename="$(find iiwa_description)/urdf/iiwa7.urdf.xacro"/>
   <!-- Properties -->
-  <xacro:property name="flex_link_mass" value="0.0001"/>
-  <xacro:property name="proximal_link_mass" value="0.0001"/>
-  <xacro:property name="distal_link_mass" value="0.0001"/>
-  <xacro:property name="proximal_pad_mass" value="0.0001"/>
-  <xacro:property name="distal_pad_mass" value="0.0001"/>
-  <xacro:property name="swivel_link_mass" value="0.0001"/>
-  <xacro:property name="base_link_mass" value="0.0074"/><!-- 0.74 -->
+  <xacro:property name="flex_link_mass" value="0.01"/>
+  <xacro:property name="proximal_link_mass" value="0.01"/>
+  <xacro:property name="distal_link_mass" value="0.01"/>
+  <xacro:property name="proximal_pad_mass" value="0.01"/>
+  <xacro:property name="distal_pad_mass" value="0.01"/>
+  <xacro:property name="swivel_link_mass" value="0.01"/>
+  <xacro:property name="base_link_mass" value="0.74"/><!-- 0.74 -->
   <xacro:property name="pad_mass" value="0.001"/>
   <!-- Parameters Limits Joints -->
   <!-- Preshape -->
-  <xacro:property name="preshape_joint_limit_effort" value="0.50"/>
-  <xacro:property name="preshape_joint_limit_velocity" value="0.5"/>
+  <xacro:property name="preshape_joint_limit_effort" value="10.0"/> <!-- 0.50 -->
+  <xacro:property name="preshape_joint_limit_velocity" value="1.0"/>
   <xacro:property name="preshape_joint_limit_lower" value="-0.00"/>
   <xacro:property name="preshape_joint_limit_upper" value="1.65"/>
   <!-- Proximal -->
-  <xacro:property name="proximal_joint_limit_effort" value="0.50"/>
-  <xacro:property name="proximal_joint_limit_velocity" value="0.5"/>
+  <xacro:property name="proximal_joint_limit_effort" value="10.0"/><!-- 0.50 -->
+  <xacro:property name="proximal_joint_limit_velocity" value="1.0"/>
   <xacro:property name="proximal_joint_limit_lower" value="0.0"/>
   <xacro:property name="proximal_joint_limit_upper" value="2.09440"/>
   <!-- Distal -->
-  <xacro:property name="distal_joint_limit_effort" value="0.50"/>
-  <xacro:property name="distal_joint_limit_velocity" value="0.5"/>
+  <xacro:property name="distal_joint_limit_effort" value="10.0"/><!-- 0.50 -->
+  <xacro:property name="distal_joint_limit_velocity" value="1.0"/>
   <xacro:property name="distal_joint_limit_lower" value="0.0"/>
   <xacro:property name="distal_joint_limit_upper" value="1.7"/>
