Commit message: trying to optimizing the grip

File: reflex_description/urdf/object_to_catch.xacro (robot description, xacro)
@@ -18,4 +18,6 @@
   <xacro:property name="rectangle_y" value="0.08"/>
   <xacro:property name="rectangle_z"   value="0.08"/>
+  <xacro:property name="mass"   value="20.5"/>
+  <!-- ${flex_length/2.0} -->
 <!-- ******************************************************************************************************* -->
 <!-- Objects to drop -->
@@ -24,5 +26,5 @@
     <inertial>
       <origin xyz="0.0 0.0 0.0"/>
-      <mass value="0.005"/>
+      <mass value="${mass}"/>
       <inertia
         ixx="0.0001" ixy="0.0" ixz="0.0"
@@ -33,5 +35,5 @@
       <origin xyz="0 0 0" rpy="0 0 0" />
       <geometry>
-        <box size="0.08 0.08 0.08"/>
+        <box size="0.08 0.20 0.08"/>
       </geometry>
       <material
@@ -44,6 +46,6 @@
         <friction>
           <ode>
-            <mu>100.0</mu>
-            <mu2>100.0</mu2>
+            <mu>1.0</mu>
+            <mu2>1.0</mu2>
           </ode>
         </friction>

File: reflex_description/urdf/reflex_takktile_2.xacro (robot description, xacro)
@@ -25,16 +25,16 @@
 <!-- Parameters Limits Joints -->
   <!-- Preshape -->
-  <xacro:property name="preshape_joint_limit_effort"     value="1.0"/>
-  <xacro:property name="preshape_joint_limit_velocity"   value="1.0"/>
+  <xacro:property name="preshape_joint_limit_effort"     value="2.0"/>
+  <xacro:property name="preshape_joint_limit_velocity"   value="0.5"/>
   <xacro:property name="preshape_joint_limit_lower"      value="-0.0872665"/>
   <xacro:property name="preshape_joint_limit_upper"      value="2.09440"/>
   <!-- Proximal -->
-  <xacro:property name="proximal_joint_limit_effort"     value="1.0"/>
-  <xacro:property name="proximal_joint_limit_velocity"   value="1.0"/>
+  <xacro:property name="proximal_joint_limit_effort"     value="2.0"/>
+  <xacro:property name="proximal_joint_limit_velocity"   value="0.5"/>
   <xacro:property name="proximal_joint_limit_lower"      value="0.0"/>
   <xacro:property name="proximal_joint_limit_upper"      value="2.09440"/>
   <!-- Distal -->
-  <xacro:property name="distal_joint_limit_effort"     value="1.0"/>
-  <xacro:property name="distal_joint_limit_velocity"   value="1.0"/>
+  <xacro:property name="distal_joint_limit_effort"     value="2.0"/>
+  <xacro:property name="distal_joint_limit_velocity"   value="0.5"/>
   <xacro:property name="distal_joint_limit_lower"      value="0.0"/>
   <xacro:property name="distal_joint_limit_upper"      value="1.8"/>

Commit message: add travis + try to add ikfast but not working yet

File: reflex_description/urdf/object_to_catch.xacro (robot description, xacro)
@@ -15,25 +15,36 @@
   <xacro:include filename="$(find iiwa_description)/urdf/iiwa7.urdf.xacro"/> -->
 <!-- Properties -->
-  <xacro:property name="rectangle_x"     value="0.08"/>
-  <xacro:property name="rectangle_y" value="0.08"/>
+  <xacro:property name="rectangle_x"     value="0.06"/>
+  <xacro:property name="rectangle_y" value="0.300"/>
   <xacro:property name="rectangle_z"   value="0.08"/>
-  <xacro:property name="mass"   value="20.5"/>
+  <xacro:property name="mass"   value="0.80"/>
   <!-- ${flex_length/2.0} -->
+<xacro:property name="I_xx"   value="${0.083333 * mass * (rectangle_y*rectangle_y + rectangle_z*rectangle_z)}"/>
+<xacro:property name="I_yy"   value="${0.083333 * mass * (rectangle_x*rectangle_x + rectangle_z*rectangle_z)}"/>
+<xacro:property name="I_zz"   value="${0.083333 * mass * (rectangle_y*rectangle_y + rectangle_x*rectangle_x)}"/>
 <!-- ******************************************************************************************************* -->
 <!-- Objects to drop -->
 <!-- ******************************************************************************************************* -->
-  <link name="square">
+  <link name="link">
     <inertial>
       <origin xyz="0.0 0.0 0.0"/>
       <mass value="${mass}"/>
       <inertia
-        ixx="0.0001" ixy="0.0" ixz="0.0"
-                         iyy="0.0001"  iyz="0.0"
-                                           izz="0.0001"/>
+        ixx="${I_xx}" ixy="0.0" ixz="0.0"
+                         iyy="${I_yy}"  iyz="0.0"
+                                           izz="${I_zz}"/>
+        <!-- <inertia
+        ixx="0.1" ixy="0.0" ixz="0.0"
+                         iyy="0.1"  iyz="0.0"
+                                           izz="0.1"/> -->
+        <!-- <inertia
+        ixx="${0.083333 * mass * (rectangle_y*rectangle_y + rectangle_z*rectangle_z)}" ixy="0.0" ixz="0.0"
+                         iyy="${0.083333 * mass * (rectangle_x*rectangle_x + rectangle_z*rectangle_z)}"  iyz="0.0"
+                                           izz="{0.083333 * mass * (rectangle_y*rectangle_y + rectangle_x*rectangle_x)}"/> -->
     </inertial>
     <visual>
       <origin xyz="0 0 0" rpy="0 0 0" />
       <geometry>
-        <box size="0.08 0.20 0.08"/>
+        <box size="${rectangle_x} ${rectangle_y} ${rectangle_z}"/>
       </geometry>
       <material
@@ -43,23 +54,33 @@
     </visual>
     <collision>
-       <surface>
+      <surface>
+        <contact>
+          <poissons_ratio>0.347</poissons_ratio>
+          <elastic_modulus>8.8e+09</elastic_modulus>
+          <ode>
+            <kp>100000</kp>
+            <kd>1</kd>
+            <max_vel>0.0</max_vel>
+            <min_depth>0.003</min_depth>
+          </ode>
+        </contact>
         <friction>
           <ode>
-            <mu>1.0</mu>
-            <mu2>1.0</mu2>
+            <mu>0.3</mu>
+            <mu2>0.3</mu2>
+            <fdir1>0 0 0</fdir1>
+            <slip1>1</slip1>
+            <slip2>1</slip2>
           </ode>
+          <!-- <torsional>
+            <coefficient>1.0</coefficient>
+            <use_patch_radius>0</use_patch_radius>
+            <surface_radius>0.05</surface_radius>
+          </torsional> -->
         </friction>
-        <!-- Change max_vel and/or min_depth to keep cones from "bouncing" -->
-        <contact>
-          <ode>
-            <!--max_vel>0</max_vel-->
-            <min_depth>0.003</min_depth>
-            <maxVel>0</maxVel>
-          </ode>
-        </contact>
       </surface>
       <origin xyz="0.0 0.0 0.0" rpy="0 0 0" />
       <geometry>
-        <box size="0.08 0.08 0.08"/>
+        <box size="${rectangle_x} ${rectangle_y} ${rectangle_z}"/>
       </geometry>
     </collision>
@@ -72,2 +93,58 @@
   </gazebo> -->
 </robot>
+<!-- <collision name='collision'>
+          <laser_retro>0</laser_retro>
+          <max_contacts>10</max_contacts>
+          <pose frame=''>0 0 0 0 -0 0</pose>
+          <geometry>
+            <mesh>
+              <uri>model://kinematics_bin/kinematics_bin.dae</uri>
+              <scale>1 1 1</scale>
+            </mesh>
+          </geometry>
+          <surface>
+            <friction>
+              <ode>
+                <mu>1</mu>
+                <mu2>1</mu2>
+                <fdir1>0 0 0</fdir1>
+                <slip1>0</slip1>
+                <slip2>0</slip2>
+              </ode>
+              <torsional>
+                <coefficient>1</coefficient>
+                <patch_radius>0</patch_radius>
+                <surface_radius>0</surface_radius>
+                <use_patch_radius>1</use_patch_radius>
+                <ode>
+                  <slip>0</slip>
+                </ode>
+              </torsional>
+            </friction>
+            <bounce>
+              <restitution_coefficient>0</restitution_coefficient>
+              <threshold>1e+06</threshold>
+            </bounce>
+            <contact>
+              <collide_without_contact>0</collide_without_contact>
+              <collide_without_contact_bitmask>1</collide_without_contact_bitmask>
+              <collide_bitmask>1</collide_bitmask>
+              <ode>
+                <soft_cfm>0</soft_cfm>
+                <soft_erp>0.2</soft_erp>
+                <kp>1e+13</kp>
+                <kd>1</kd>
+                <max_vel>0.01</max_vel>
+                <min_depth>0</min_depth>
+              </ode>
+              <bullet>
+                <split_impulse>1</split_impulse>
+                <split_impulse_penetration_threshold>-0.01</split_impulse_penetration_threshold>
+                <soft_cfm>0</soft_cfm>
+                <soft_erp>0.2</soft_erp>
+                <kp>1e+13</kp>
+                <kd>1</kd>
+              </bullet>
+            </contact>
+          </surface>
+</collision> -->

File: reflex_description/urdf/reflex.gazebo.xacro (robot description, xacro)
@@ -107,3 +107,142 @@
 			<!-- <maxContacts>1</maxContacts> -->
   </gazebo>
+  <!-- Add gazebo - pkg for grasping -->
+  <!-- <gazebo>
+   <plugin name="gazebo_grasp_fix" filename="libgazebo_grasp_fix.so">
+        <arm>
+           <arm_name>base_link</arm_name>
+           <palm_link>pad</palm_link>
+           <gripper_link>distal_pad_1</gripper_link>
+           <gripper_link>distal_pad_2</gripper_link>
+           <gripper_link>distal_pad_3</gripper_link>
+           <gripper_link>proximal_pad_1</gripper_link>
+           <gripper_link>proximal_pad_2</gripper_link>
+           <gripper_link>proximal_pad_3</gripper_link>
+        </arm>
+       <forces_angle_tolerance>100</forces_angle_tolerance>
+       <update_rate>4</update_rate>
+       <grip_count_threshold>4</grip_count_threshold>
+       <max_grip_count>8</max_grip_count>
+       <release_tolerance>0.005</release_tolerance>
+       <disable_collisions_on_attach>false</disable_collisions_on_attach>
+       <contact_topic>__default_topic__</contact_topic>
+    </plugin>
+  </gazebo> -->
+  <!-- <gazebo>
+   <plugin name="gazebo_grasp_fix" filename="libgazebo_grasp_fix.so">
+        <arm>
+           <arm_name>base_link</arm_name>
+           <palm_link>pad</palm_link>
+           <gripper_link>iiwa/distal_pad_1</gripper_link>
+           <gripper_link>iiwa/distal_pad_2</gripper_link>
+           <gripper_link>iiwa/distal_pad_3</gripper_link>
+           <gripper_link>iiwa/proximal_pad_1</gripper_link>
+           <gripper_link>iiwa/proximal_pad_2</gripper_link>
+           <gripper_link>iiwa/proximal_pad_3</gripper_link>
+        </arm>
+       <forces_angle_tolerance>100</forces_angle_tolerance>
+       <update_rate>10</update_rate>
+       <grip_count_threshold>2</grip_count_threshold>
+       <max_grip_count>10</max_grip_count>
+       <release_tolerance>0.005</release_tolerance>
+       <disable_collisions_on_attach>true</disable_collisions_on_attach>
+       <contact_topic>__default_topic__</contact_topic>
+    </plugin>
+  </gazebo> -->
+  <gazebo>
+   <plugin name="gazebo_grasp_fix" filename="libgazebo_grasp_fix.so">
+        <arm>
+          <arm_name>arm_name_default_john</arm_name>
+          <palm_link>iiwa_link_7</palm_link>
+          <gripper_link>distal_1</gripper_link>
+          <gripper_link>distal_2</gripper_link>
+          <gripper_link>distal_3</gripper_link>
+          <gripper_link>proximal_1</gripper_link>
+          <gripper_link>proximal_2</gripper_link>
+          <gripper_link>proximal_3</gripper_link>
+          <gripper_link>proximal_1_sensor_1</gripper_link>
+          <gripper_link>proximal_1_sensor_2</gripper_link>
+          <gripper_link>proximal_1_sensor_3</gripper_link>
+          <gripper_link>proximal_1_sensor_4</gripper_link>
+          <gripper_link>proximal_1_sensor_5</gripper_link>
+          <gripper_link>proximal_2_sensor_1</gripper_link>
+          <gripper_link>proximal_2_sensor_2</gripper_link>
+          <gripper_link>proximal_2_sensor_3</gripper_link>
+          <gripper_link>proximal_2_sensor_4</gripper_link>
+          <gripper_link>proximal_2_sensor_5</gripper_link>
+          <gripper_link>proximal_3_sensor_1</gripper_link>
+          <gripper_link>proximal_3_sensor_2</gripper_link>
+          <gripper_link>proximal_3_sensor_3</gripper_link>
+          <gripper_link>proximal_3_sensor_4</gripper_link>
+          <gripper_link>proximal_3_sensor_5</gripper_link>
+          <gripper_link>distal_1_sensor_1</gripper_link>
+          <gripper_link>distal_1_sensor_2</gripper_link>
+          <gripper_link>distal_1_sensor_3</gripper_link>
+          <gripper_link>distal_1_sensor_4</gripper_link>
+          <gripper_link>distal_2_sensor_1</gripper_link>
+          <gripper_link>distal_2_sensor_2</gripper_link>
+          <gripper_link>distal_2_sensor_3</gripper_link>
+          <gripper_link>distal_2_sensor_4</gripper_link>
+          <gripper_link>distal_3_sensor_1</gripper_link>
+          <gripper_link>distal_3_sensor_2</gripper_link>
+          <gripper_link>distal_3_sensor_3</gripper_link>
+          <gripper_link>distal_3_sensor_4</gripper_link>
+        </arm>
+      <forces_angle_tolerance>90</forces_angle_tolerance>
+      <update_rate>100</update_rate>
+      <grip_count_threshold>6</grip_count_threshold>
+      <max_grip_count>20</max_grip_count>
+      <release_tolerance>0.05</release_tolerance>
+      <disable_collisions_on_attach>true</disable_collisions_on_attach>
+      <contact_topic>__default_topic__</contact_topic>
+    </plugin>
+  </gazebo>
+  <!-- <gazebo>
+   <plugin name="gazebo_grasp_fix" filename="libgazebo_grasp_fix.so">
+        <arm>
+          <arm_name>base_link</arm_name>
+          <palm_link>iiwa/pad</palm_link>
+          <gripper_link>iiwa/distal_1</gripper_link>
+          <gripper_link>iiwa/distal_2</gripper_link>
+          <gripper_link>iiwa/distal_3</gripper_link>
+          <gripper_link>iiwa/proximal_1</gripper_link>
+          <gripper_link>iiwa/proximal_2</gripper_link>
+          <gripper_link>iiwa/proximal_3</gripper_link>
+          <gripper_link>iiwa/proximal_1_sensor_1</gripper_link>
+          <gripper_link>iiwa/proximal_1_sensor_2</gripper_link>
+          <gripper_link>iiwa/proximal_1_sensor_3</gripper_link>
+          <gripper_link>iiwa/proximal_1_sensor_4</gripper_link>
+          <gripper_link>iiwa/proximal_1_sensor_5</gripper_link>
+          <gripper_link>iiwa/proximal_2_sensor_1</gripper_link>
+          <gripper_link>iiwa/proximal_2_sensor_2</gripper_link>
+          <gripper_link>iiwa/proximal_2_sensor_3</gripper_link>
+          <gripper_link>iiwa/proximal_2_sensor_4</gripper_link>
+          <gripper_link>iiwa/proximal_2_sensor_5</gripper_link>
+          <gripper_link>iiwa/proximal_3_sensor_1</gripper_link>
+          <gripper_link>iiwa/proximal_3_sensor_2</gripper_link>
+          <gripper_link>iiwa/proximal_3_sensor_3</gripper_link>
+          <gripper_link>iiwa/proximal_3_sensor_4</gripper_link>
+          <gripper_link>iiwa/proximal_3_sensor_5</gripper_link>
+          <gripper_link>iiwa/distal_1_sensor_1</gripper_link>
+          <gripper_link>iiwa/distal_1_sensor_2</gripper_link>
+          <gripper_link>iiwa/distal_1_sensor_3</gripper_link>
+          <gripper_link>iiwa/distal_1_sensor_4</gripper_link>
+          <gripper_link>iiwa/distal_2_sensor_1</gripper_link>
+          <gripper_link>iiwa/distal_2_sensor_2</gripper_link>
+          <gripper_link>iiwa/distal_2_sensor_3</gripper_link>
+          <gripper_link>iiwa/distal_2_sensor_4</gripper_link>
+          <gripper_link>iiwa/distal_3_sensor_1</gripper_link>
+          <gripper_link>iiwa/distal_3_sensor_2</gripper_link>
+          <gripper_link>iiwa/distal_3_sensor_3</gripper_link>
+          <gripper_link>iiwa/distal_3_sensor_4</gripper_link>
+        </arm>
+      <forces_angle_tolerance>180</forces_angle_tolerance>
+      <update_rate>100</update_rate>
+      <grip_count_threshold>2</grip_count_threshold>
+      <max_grip_count>10</max_grip_count>
+      <release_tolerance>0.05</release_tolerance>
+      <disable_collisions_on_attach>true</disable_collisions_on_attach>
+      <contact_topic>__default_topic__</contact_topic>
+    </plugin>
+  </gazebo> -->
 </robot>
