Commit message: add travis + try to add ikfast but not working yet

File: reflex_description/urdf/reflex_takktile_2.xacro (robot description, xacro)
@@ -5,6 +5,7 @@
           - Create the macro of simplifying creation of the repetitive part
    -->
-<robot name="reflex_takktile_2" xmlns:xacro="http://ros.org/wiki/xacro">
-<!-- Incudes -->
+<robot name="reflex_takktile_2"
+  xmlns:xacro="http://ros.org/wiki/xacro">
+  <!-- Incudes -->
   <!-- <xacro:include filename="$(find reflex_description)/urdf/reflex_takktile_2.xacro" />   -->
   <xacro:include filename="$(find reflex_description)/urdf/reflex.transmission.xacro" />
@@ -14,32 +15,32 @@
   <xacro:include filename="$(find iiwa_description)/urdf/iiwa7.xacro"/>
   <xacro:include filename="$(find iiwa_description)/urdf/iiwa7.urdf.xacro"/>
-<!-- Properties -->
-  <xacro:property name="flex_link_mass"     value="0.01"/>
+  <!-- Properties -->
+  <xacro:property name="flex_link_mass" value="0.01"/>
   <xacro:property name="proximal_link_mass" value="0.01"/>
-  <xacro:property name="distal_link_mass"   value="0.01"/>
-  <xacro:property name="proximal_pad_mass"  value="0.01"/>
-  <xacro:property name="distal_pad_mass"    value="0.01"/>
-  <xacro:property name="swivel_link_mass"   value="0.01"/>
-  <xacro:property name="base_link_mass"     value="0.74"/>
-  <xacro:property name="pad_mass"           value="0.1"/>
-<!-- Parameters Limits Joints -->
+  <xacro:property name="distal_link_mass" value="0.01"/>
+  <xacro:property name="proximal_pad_mass" value="0.01"/>
+  <xacro:property name="distal_pad_mass" value="0.01"/>
+  <xacro:property name="swivel_link_mass" value="0.01"/>
+  <xacro:property name="base_link_mass" value="0.34"/><!-- 0.74 -->
+  <xacro:property name="pad_mass" value="0.1"/>
+  <!-- Parameters Limits Joints -->
   <!-- Preshape -->
-  <xacro:property name="preshape_joint_limit_effort"     value="2.0"/>
-  <xacro:property name="preshape_joint_limit_velocity"   value="0.5"/>
-  <xacro:property name="preshape_joint_limit_lower"      value="-0.0872665"/>
-  <xacro:property name="preshape_joint_limit_upper"      value="2.09440"/>
+  <xacro:property name="preshape_joint_limit_effort" value="0.50"/>
+  <xacro:property name="preshape_joint_limit_velocity" value="0.5"/>
+  <xacro:property name="preshape_joint_limit_lower" value="-0.00"/>
+  <xacro:property name="preshape_joint_limit_upper" value="1.65"/>
   <!-- Proximal -->
-  <xacro:property name="proximal_joint_limit_effort"     value="2.0"/>
-  <xacro:property name="proximal_joint_limit_velocity"   value="0.5"/>
-  <xacro:property name="proximal_joint_limit_lower"      value="0.0"/>
-  <xacro:property name="proximal_joint_limit_upper"      value="2.09440"/>
+  <xacro:property name="proximal_joint_limit_effort" value="0.50"/>
+  <xacro:property name="proximal_joint_limit_velocity" value="0.5"/>
+  <xacro:property name="proximal_joint_limit_lower" value="0.0"/>
+  <xacro:property name="proximal_joint_limit_upper" value="2.09440"/>
   <!-- Distal -->
-  <xacro:property name="distal_joint_limit_effort"     value="2.0"/>
-  <xacro:property name="distal_joint_limit_velocity"   value="0.5"/>
-  <xacro:property name="distal_joint_limit_lower"      value="0.0"/>
-  <xacro:property name="distal_joint_limit_upper"      value="1.8"/>
-<!-- ################ ################ ################ ################ ################ ################ -->
-<!-- ################ XACRO PORTION OF THE URDF, FOR MAKING THE FLEXIBLE JOINTS ################ -->
-<!-- ################ ################ ################ ################ ################ ################ -->
+  <xacro:property name="distal_joint_limit_effort" value="0.50"/>
+  <xacro:property name="distal_joint_limit_velocity" value="0.5"/>
+  <xacro:property name="distal_joint_limit_lower" value="0.0"/>
+  <xacro:property name="distal_joint_limit_upper" value="1.7"/>
+  <!-- ################ ################ ################ ################ ################ ################ -->
+  <!-- ################ XACRO PORTION OF THE URDF, FOR MAKING THE FLEXIBLE JOINTS ################ -->
+  <!-- ################ ################ ################ ################ ################ ################ -->
   <xacro:property name="flex_length" value="0.016" />
   <xacro:property name="distal_length" value="0.050" />
@@ -47,9 +48,9 @@
   <xacro:property name="prox_length" value="0.060" />
   <xacro:property name="pi" value="3.1415" />
-<!-- ################ ################ ################ ################ ################ ################ -->
-<!-- ################ THE SECTION CREATED BY SOLIDWORKS EXPORTER, CUT AND PASTE THIS IN HERE ################ -->
-<!-- ################ YOU CAN ALTER THE COLORS FROM HERE ################ -->
-<!-- ################ COMMENT OUT ALL dist*_joint PIECES OF THIS URDF SO THE FLEX JOINTS CAN LINK UP ################ -->
-<!-- ################ ################ ################ ################ ################ ################ -->
+  <!-- ################ ################ ################ ################ ################ ################ -->
+  <!-- ################ THE SECTION CREATED BY SOLIDWORKS EXPORTER, CUT AND PASTE THIS IN HERE ################ -->
+  <!-- ################ YOU CAN ALTER THE COLORS FROM HERE ################ -->
+  <!-- ################ COMMENT OUT ALL dist*_joint PIECES OF THIS URDF SO THE FLEX JOINTS CAN LINK UP ################ -->
+  <!-- ################ ################ ################ ################ ################ ################ -->
   <link name="base_link">
     <inertial>
@@ -58,21 +59,17 @@
       <!-- TODO: CALCULATES THE MASS AND INERTIAs -->
       <mass value="${base_link_mass}"/>
-      <inertia
-        ixx="0.0001" ixy="0.0" ixz="0.0"
-                         iyy="0.0001"  iyz="0.0"
-                                           izz="0.0001"/>
+      <inertia ixx="0.0001" ixy="0.0" ixz="0.0" iyy="0.0001" iyz="0.0" izz="0.0001"/>
     </inertial>
     <!-- TODO: Change the BASE OF the hand to the version 2 -->
     <visual>
-      <origin
-        xyz="0 0 0" rpy="0 0 0" />
-      <geometry>
-        <mesh
-          filename="package://reflex_description/meshes/base_link.STL" />
-      </geometry>
-      <material
-        name="base_color">
+      <origin xyz="0 0 0" rpy="0 0 0" />
+      <geometry>
+        <!-- <mesh filename="$(find reflex_description)/meshes/base_link.stl" /> -->
+         <mesh filename="package://reflex_description/meshes/base_link.stl" />
+         <!-- <mesh filename="package://iiwa_description/meshes/iiwa7/visual/link_0.stl"/> -->
+      </geometry>
+      <!-- <material name="base_color">
         <xacro:base_color/>
-      </material>
+      </material> -->
     </visual>
     <!-- TODO: Change the BASE OF the hand to the version 2 -->
@@ -80,5 +77,5 @@
       <origin xyz="0.0 0.0 0.0" rpy="0 0 0" />
       <geometry>
-        <mesh filename="package://reflex_description/meshes/base_link.STL" />
+        <mesh filename="package://reflex_description/meshes/base_link.stl" />
       </geometry>
     </collision>
@@ -86,7 +83,7 @@
   <!-- For a tool on a arm, uncomment this part -->
   <joint name="tool_joint" type="fixed">
-      <parent link="iiwa_link_ee" />
-      <child link = "base_link" />
-      <origin xyz="0.0 0.0 0.0" rpy="0 0.0 3.14159" />
+    <parent link="iiwa_link_ee" />
+    <child link = "base_link" />
+    <origin xyz="0.0 0.0 0.0" rpy="0 0.0 3.14159" />
   </joint>
   <link name="pad">
@@ -96,54 +93,41 @@
       <!-- TODO: CALCULATES THE MASS AND INERTIAs -->
       <mass value="0.1"/>
-      <inertia
-        ixx="0.0001" ixy="0.0" ixz="0.0"
-                         iyy="0.0001"  iyz="0.0"
-                                           izz="0.0001"/>
+      <inertia ixx="0.0001" ixy="0.0" ixz="0.0" iyy="0.0001" iyz="0.0" izz="0.0001"/>
     </inertial>
     <visual>
       <origin xyz="0 0 0" rpy="0 0 0" />
       <geometry>
-        <mesh
-          filename="package://reflex_description/meshes/pad.STL" />
-      </geometry>
-      <material
-        name="">
-        <xacro:pad_color/>
-      </material>
+        <mesh filename="package://reflex_description/meshes/pad.stl" />
+      </geometry>
+      <!-- <material name="">
+        <xacro:pad/>
+      </material> -->
     </visual>
     <collision>
       <origin xyz="0.0 0.0 0.0" rpy="0 0 0" />
       <geometry>
-        <mesh filename="package://reflex_description/meshes/pad.STL" />
+        <mesh filename="package://reflex_description/meshes/pad.stl" />
       </geometry>
     </collision>
   </link>
   <joint name="pad_joint" type="fixed">
-    <origin
-      xyz="0.02 0 0.063"
-      rpy="1.5707963267949 5.55111512312578E-17 -1.5707963267949" />
-    <parent
-      link="base_link" />
-    <child
-      link="pad" />
-    <axis
-      xyz="0 0 0" />
+    <origin xyz="0.02 0 0.063" rpy="1.5707963267949 5.55111512312578E-17 -1.5707963267949" />
+    <parent link="base_link" />
+    <child link="pad" />
+    <axis xyz="0 0 0" />
   </joint>
   <!-- Add the tool tips which is the pose of the hand effector -->
   <!-- TODO Check the offset of the tool! -->
   <joint name="tool_ee_joint" type="fixed">
-  <parent link="base_link" />
-  <child link = "tool_link_ee" />
-  <origin xyz="0 0 0.1275" rpy="0 ${0.0/1.0} 0" />
-</joint>
-<!--  The TCP frame is here defined -->
-<link name="tool_link_ee">
-  <!-- <inertial>
+    <parent link="base_link" />
+    <child link = "tool_link_ee" />
+    <origin xyz="0 0 0.1275" rpy="0 ${0.0/1.0} 0" />
+  </joint>
+  <!--  The TCP frame is here defined -->
+  <link name="tool_link_ee">
+    <!-- <inertial>
     <origin xyz="0.0 0.0 0.0"/>
     <mass value="0.0001"/>
-    <inertia
-      ixx="0.0001" ixy="0.0" ixz="0.0"
-                        iyy="0.0001"  iyz="0.0"
-                                          izz="0.0001"/>
+    <inertia ixx="0.0001" ixy="0.0" ixz="0.0" iyy="0.0001" iyz="0.0" izz="0.0001"/>
   </inertial>
   <visual>
@@ -152,6 +136,5 @@
      <cylinder length="${length}" radius="${radius}"/>
     </geometry>
-    <material
-      name="">
+    <material name="">
       <xacro:pad_color/>
     </material>
@@ -163,6 +146,6 @@
     </geometry>
   </collision> -->
-</link>
-<!-- *****************************************FINGER 1**************************************************** -->
+  </link>
+  <!-- *****************************************FINGER 1**************************************************** -->
   <link name="swivel_1">
     <inertial>
@@ -171,39 +154,29 @@
       <!-- TODO: CALCULATES THE MASS AND INERTIAs -->
       <mass value="0.01"/>
-      <inertia
-        ixx="0.0001" ixy="0.0" ixz="0.0"
-                         iyy="0.0001"  iyz="0.0"
-                                           izz="0.0001"/>
+      <inertia ixx="0.0001" ixy="0.0" ixz="0.0" iyy="0.0001" iyz="0.0" izz="0.0001"/>
     </inertial>
     <visual>
       <origin xyz="0 0 0" rpy="0 0 0" />
       <geometry>
-        <mesh
-          filename="package://reflex_description/meshes/swivel_1.STL" />
-      </geometry>
-      <material
-        name="">
+        <mesh filename="package://reflex_description/meshes/swivel_1.stl" />
+      </geometry>
+      <!-- <material name="">
         <xacro:swivel_color/>
-      </material>
+      </material> -->
     </visual>
     <collision>
       <origin xyz="0.0 0.0 0.0" rpy="0 0 0" />
       <geometry>
-        <mesh filename="package://reflex_description/meshes/swivel_1.STL" />
+        <mesh filename="package://reflex_description/meshes/swivel_1.stl" />
       </geometry>
     </collision>
   </link>
   <joint name="preshape_1" type="revolute">
-    <origin
-      xyz="0.0503973683071414 -0.026 0.063"
-      rpy="6.75550818663469E-16 1.97993848419069E-16 -2.77555756156289E-16" />
+    <origin xyz="0.0503973683071414 -0.026 0.063" rpy="6.75550818663469E-16 1.97993848419069E-16 -2.77555756156289E-16" />
     <parent link="base_link" />
     <child link="swivel_1" />
     <axis xyz="0 0 -1" />
     <!-- <limit effort="30" velocity="1.0" lower="-0.0872665" upper="2.0944" /> -->
-    <limit effort="${preshape_joint_limit_effort}"
-            velocity="${preshape_joint_limit_velocity}"
-            lower="${preshape_joint_limit_lower}"
-            upper="${preshape_joint_limit_upper}" />
+    <limit effort="${preshape_joint_limit_effort}" velocity="${preshape_joint_limit_velocity}" lower="${preshape_joint_limit_lower}" upper="${preshape_joint_limit_upper}" />
   </joint>
   <link name="proximal_1">
@@ -213,38 +186,28 @@
       <!-- TODO: CALCULATES THE MASS AND INERTIAs -->
       <mass value="0.01"/>
-      <inertia
-        ixx="0.0001" ixy="0.0" ixz="0.0"
-                         iyy="0.0001"  iyz="0.0"
-                                           izz="0.0001"/>
+      <inertia ixx="0.0001" ixy="0.0" ixz="0.0" iyy="0.0001" iyz="0.0" izz="0.0001"/>
     </inertial>
     <visual>
       <origin xyz="-0.011 0.007 0.011" rpy="3.1459 0 0"/>
       <geometry>
-        <mesh
-          filename="package://reflex_description/meshes/proximal_1.STL" />
-      </geometry>
-      <material
-        name="">
+        <mesh filename="package://reflex_description/meshes/proximal_1.stl" />
+      </geometry>
+      <!-- <material name="">
         <xacro:proximal_color/>
-      </material>
+      </material> -->
     </visual>
     <collision>
       <origin xyz="-0.011 0.007 0.011" rpy="3.1459 0 0" />
       <geometry>
-        <mesh filename="package://reflex_description/meshes/proximal_1.STL" />
+        <mesh filename="package://reflex_description/meshes/proximal_1.stl" />
       </geometry>
     </collision>
   </link>
   <joint name="proximal_joint_1" type="revolute">
-    <origin
-      xyz="0.01 0 0.0186"
-      rpy="-6.20039667432211E-16 0.05 2.22044604925031E-16" />
+    <origin xyz="0.01 0 0.0186" rpy="-6.20039667432211E-16 0.05 2.22044604925031E-16" />
     <parent link="swivel_1" />
     <child link="proximal_1" />
     <axis xyz="0 -1 0" />
-    <limit effort="${proximal_joint_limit_effort}"
-            velocity="${proximal_joint_limit_velocity}"
-            lower="${proximal_joint_limit_lower}"
-            upper="${proximal_joint_limit_upper}" />
+    <limit effort="${proximal_joint_limit_effort}" velocity="${proximal_joint_limit_velocity}" lower="${proximal_joint_limit_lower}" upper="${proximal_joint_limit_upper}" />
   </joint>
   <link name="proximal_pad_1">
@@ -254,21 +217,14 @@
       <!-- TODO: CALCULATES THE MASS AND INERTIAs -->
       <mass value="0.01"/>
-      <inertia
-        ixx="0.0001"  ixy="0.0"     ixz="0.0"
-                      iyy="0.0001"  iyz="0.0"
-                                    izz="0.0001"/>
-    </inertial>
-    <visual>
-      <origin
-        xyz="-0.008 0.014 -0.002"
-        rpy="1.5708 1.5708 0" />
-      <geometry>
-        <mesh
-          filename="package://reflex_description/meshes/proximal_pad_1.STL" />
-      </geometry>
-      <material
-        name="">
+      <inertia ixx="0.0001" ixy="0.0" ixz="0.0" iyy="0.0001" iyz="0.0" izz="0.0001"/>
+    </inertial>
+    <visual>
+      <origin xyz="-0.008 0.014 -0.002" rpy="1.5708 1.5708 0" />
+      <geometry>
+        <mesh filename="package://reflex_description/meshes/proximal_pad_1.stl" />
+      </geometry>
+      <!-- <material name="">
         <xacro:pad_color/>
-      </material>
+      </material> -->
     </visual>
     <!-- Keep for souvenir -->
@@ -276,5 +232,5 @@
       <origin xyz="-0.008 0.014 -0.002" rpy="1.5708 1.5708 0" />
       <geometry>
-        <mesh filename="package://reflex_description/meshes/proximal_pad_1.STL" />
+        <mesh filename="package://reflex_description/meshes/proximal_pad_1.stl" />
       </geometry>
     </collision> -->
@@ -282,5 +238,5 @@
       <origin xyz="-0.008 0.014 -0.002" rpy="1.5708 1.5708 0" />
       <geometry>
-        <mesh filename="package://reflex_description/meshes/proximal_pad_1.STL" />
+        <mesh filename="package://reflex_description/meshes/proximal_pad_1.stl" />
       </geometry>
     </collision>
@@ -293,31 +249,27 @@
   </joint>
   <link name="flex_link_1">
-     <inertial>
-      <!-- TODO: CALCULATES CENTER OF MASS -->
-      <origin xyz="0.0 0.0 0.0"/>
-      <!-- TODO: CALCULATES THE MASS AND INERTIAs -->
-      <mass value="0.01"/>
-      <inertia
-        ixx="0.0001"  ixy="0.0"     ixz="0.0"
-                      iyy="0.0001"  iyz="0.0"
-                                    izz="0.0001"/>
-    </inertial>
-    <visual>
-        <!-- <origin xyz="${flex_length/2.0} -0.008 0.001" rpy="${pi/2} 0 ${pi/2}" /> -->
-        <origin xyz="${flex_length/2.0} 0.0 0.0" rpy="0.0 0.0 0.0" />
-        <geometry>
-          <!-- <mesh filename="package://reflex_description/meshes/flex_block.STL" /> -->
-          <box size="${flex_length*1.0} 0.014 0.006"/>
-        </geometry>
-        <material
-          name="">
-          <xacro:flex_color/>
-        </material>
-      </visual>
-    <collision>
+    <inertial>
+      <!-- TODO: CALCULATES CENTER OF MASS -->
+      <origin xyz="0.0 0.0 0.0"/>
+      <!-- TODO: CALCULATES THE MASS AND INERTIAs -->
+      <mass value="0.01"/>
+      <inertia ixx="0.0001" ixy="0.0" ixz="0.0" iyy="0.0001" iyz="0.0" izz="0.0001"/>
+    </inertial>
+    <visual>
       <!-- <origin xyz="${flex_length/2.0} -0.008 0.001" rpy="${pi/2} 0 ${pi/2}" /> -->
       <origin xyz="${flex_length/2.0} 0.0 0.0" rpy="0.0 0.0 0.0" />
       <geometry>
-        <!-- <mesh filename="package://reflex_description/meshes/flex_block.STL" /> -->
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
File: reflex_description/urdf/tactile_sensors.xacro (robot description, xacro)
@@ -13,4 +13,9 @@
     <xacro:property name="distal_offset_z"   value="0.010"/>
     <xacro:property name="number_separation_distal"   value="5.0"/>
+    <xacro:property name="flex_length" value="0.016" />
+    <xacro:property name="distal_length" value="0.050" />
+    <xacro:property name="num_steps" value="9" />
+    <xacro:property name="prox_length" value="0.060" />
+    <xacro:property name="pi" value="3.1415" />
     <!-- Sensors parameters -->
     <xacro:property name="radius"   value="0.003"/>
@@ -31,8 +36,8 @@
                 <cylinder length="${length}" radius="${radius}"/>
             </geometry>
-            <material
-                name="">
-                <xacro:pad_color/>
-            </material>
+            <!-- <material
+                name="">
+                <xacro:pad_color/>
+            </material> -->
             </visual>
             <collision name="proximal_${finger_number}_sensor_1_collision">
@@ -63,8 +68,8 @@
                 <cylinder length="${length}" radius="${radius}"/>
             </geometry>
-            <material
-                name="">
-                <xacro:pad_color/>
-            </material>
+            <!-- <material
+                name="">
+                <xacro:pad_color/>
+            </material> -->
             </visual>
             <collision name="proximal_${finger_number}_sensor_2_collision">
@@ -95,8 +100,8 @@
                 <cylinder length="${length}" radius="${radius}"/>
             </geometry>
-            <material
-                name="">
-                <xacro:pad_color/>
-            </material>
+            <!-- <material
+                name="">
+                <xacro:pad_color/>
+            </material> -->
             </visual>
             <collision name="proximal_${finger_number}_sensor_3_collision">
@@ -127,8 +132,8 @@
                 <cylinder length="${length}" radius="${radius}"/>
             </geometry>
-            <material
-                name="">
-                <xacro:pad_color/>
-            </material>
+            <!-- <material
+                name="">
+                <xacro:pad_color/>
+            </material> -->
             </visual>
             <collision name="proximal_${finger_number}_sensor_4_collision">
@@ -159,8 +164,8 @@
                 <cylinder length="${length}" radius="${radius}"/>
             </geometry>
-            <material
-                name="">
-                <xacro:pad_color/>
-            </material>
+            <!-- <material
+                name="">
+                <xacro:pad_color/>
+            </material> -->
             </visual>
             <collision name="proximal_${finger_number}_sensor_5_collision">
@@ -193,8 +198,8 @@
                 <cylinder length="${length}" radius="${radius}"/>
             </geometry>
-            <material
-                name="">
-                <xacro:pad_color/>
-            </material>
+            <!-- <material
+                name="">
+                <xacro:pad_color/>
+            </material> -->
             </visual>
             <collision name="distal_${finger_number}_sensor_1_collision">
@@ -225,8 +230,8 @@
                 <cylinder length="${length}" radius="${radius}"/>
             </geometry>
-            <material
-                name="">
-                <xacro:pad_color/>
-            </material>
+            <!-- <material
+                name="">
+                <xacro:pad_color/>
+            </material> -->
             </visual>
             <collision name="distal_${finger_number}_sensor_2_collision">
@@ -257,8 +262,8 @@
                 <cylinder length="${length}" radius="${radius}"/>
             </geometry>
-            <material
-                name="">
-                <xacro:pad_color/>
-            </material>
+            <!-- <material
+                name="">
+                <xacro:pad_color/>
+            </material> -->
             </visual>
             <collision name="distal_${finger_number}_sensor_3_collision">
@@ -289,8 +294,8 @@
                 <cylinder length="${length}" radius="${radius}"/>
             </geometry>
-            <material
-                name="">
-                <xacro:pad_color/>
-            </material>
+            <!-- <material
+                name="">
+                <xacro:pad_color/>
+            </material> -->
             </visual>
             <collision name="distal_${finger_number}_sensor_4_collision">
