Commit message: add .

File: reflex_description/urdf/object_to_catch.xacro (robot description, xacro)
@@ -18,5 +18,5 @@
   <xacro:property name="rectangle_y" value="0.20"/>
   <xacro:property name="rectangle_z"   value="0.08"/>
-  <xacro:property name="mass"   value="0.80"/>
+  <xacro:property name="mass"   value="0.30"/>
   <!-- ${flex_length/2.0} -->
 <xacro:property name="I_xx"   value="${0.083333 * mass * (rectangle_y*rectangle_y + rectangle_z*rectangle_z)}"/>
@@ -55,6 +55,6 @@
         <friction>
           <ode>
-            <mu>0.3</mu>
-            <mu2>0.3</mu2>
+            <mu>0.1</mu>
+            <mu2>0.1</mu2>
             <fdir1>0 0 0</fdir1>
             <slip1>1</slip1>

File: reflex_description/urdf/reflex_takktile_2.xacro (robot description, xacro)
@@ -26,16 +26,16 @@
   <!-- Parameters Limits Joints -->
   <!-- Preshape -->
-  <xacro:property name="preshape_joint_limit_effort" value="10.0"/> <!-- 0.50 -->
-  <xacro:property name="preshape_joint_limit_velocity" value="1.0"/>
+  <xacro:property name="preshape_joint_limit_effort" value="100.0"/> <!-- 0.50 -->
+  <xacro:property name="preshape_joint_limit_velocity" value="10.0"/>
   <xacro:property name="preshape_joint_limit_lower" value="-0.00"/>
   <xacro:property name="preshape_joint_limit_upper" value="1.65"/>
   <!-- Proximal -->
-  <xacro:property name="proximal_joint_limit_effort" value="10.0"/><!-- 0.50 -->
-  <xacro:property name="proximal_joint_limit_velocity" value="1.0"/>
+  <xacro:property name="proximal_joint_limit_effort" value="100.0"/><!-- 0.50 -->
+  <xacro:property name="proximal_joint_limit_velocity" value="10.0"/>
   <xacro:property name="proximal_joint_limit_lower" value="0.0"/>
   <xacro:property name="proximal_joint_limit_upper" value="2.09440"/>
   <!-- Distal -->
-  <xacro:property name="distal_joint_limit_effort" value="10.0"/><!-- 0.50 -->
-  <xacro:property name="distal_joint_limit_velocity" value="1.0"/>
+  <xacro:property name="distal_joint_limit_effort" value="51000.0"/><!-- 0.50 -->
+  <xacro:property name="distal_joint_limit_velocity" value="10.0"/>
   <xacro:property name="distal_joint_limit_lower" value="0.0"/>
   <xacro:property name="distal_joint_limit_upper" value="1.7"/>
